File: Wasp_Hive.kicad_pcb (KiCad board)
At the start: 2 copper layers, 147 parts, among them J0 WASP_OUT, J1 WASP_OUT, J10 WASP_OUT, J11 WASP_OUT, J12 WASP_OUT, J13 WASP_OUT, J14 WASP_OUT, J15 WASP_OUT, J16 FM_IN, J17 DENS_IN, J18 DENS_IN, J2 WASP_OUT, J3 WASP_OUT, J4 WASP_OUT, J5 WASP_OUT, J6 WASP_OUT, J7 WASP_OUT, J8 WASP_OUT, J9 WASP_OUT, Q1 MMBT3904, Q2 MMBT3904, U0 74HC245, U1 74HC245, U2 MCP6002-xP, U3 L78M05ABDT-TR, U4 MCP6002-xP, U5 TEENSY_3.2_MINIMAL

Commit message: first form factor
Parts:
- removed C1: 0.33uf, Capacitor_SMD:C_0603_1608Metric_Pad1.05x0.95mm_HandSolder_SmallRef
- removed C2: 0.1uf, Capacitor_SMD:C_0603_1608Metric_Pad1.05x0.95mm_HandSolder_SmallRef
- removed D32, D33, D34, D35: SM4007PL, Diode_SMD:D_SOD-123
- removed Q1, Q2: MMBT3904, Package_TO_SOT_SMD:SOT-23
- removed R0, R12, R15, R18, R21, R24, R27, R3, R30, R33, R36, R39, R42, R45, R6, R9: LRV_R, Resistor_SMD:R_0603_1608Metric_Pad1.05x0.95mm_HandSolder_SmallRef
- removed R1, R10, R13, R16, R19, R22, R25, R28, R31, R34, R37, R4, R40, R43, R46, R7: WSP_R, Resistor_SMD:R_0603_1608Metric_Pad1.05x0.95mm_HandSolder_SmallRef
- removed R11, R14, R17, R2, R20, R23, R26, R29, R32, R35, R38, R41, R44, R47, R5, R8: O_R, Resistor_SMD:R_0603_1608Metric_Pad1.05x0.95mm_HandSolder_SmallRef
- removed R48, R49, R51, R52, R53, R54: 100k, Resistor_SMD:R_0603_1608Metric_Pad1.05x0.95mm_HandSolder_SmallRef
- removed R50: 1k, Resistor_SMD:R_0603_1608Metric_Pad1.05x0.95mm_HandSolder_SmallRef
- removed the REF** at (78.0, 160.0)
- removed the REF** at (68.0, 143.0)
- removed the REF** at (48.0, 143.0)
- removed the REF** at (28.0, 143.0)
- removed the REF** at (58.0, 126.0)
- removed the REF** at (48.0, 109.0)
- removed the REF** at (58.0, 92.0)
- removed the REF** at (38.0, 126.0)
- removed the REF** at (28.0, 109.0)
- removed the REF** at (68.0, 75.0)
- removed the REF** at (48.0, 75.0)
- removed the REF** at (68.0, 109.0)
- removed the REF** at (38.0, 92.0)
- removed the REF** at (58.0, 160.0)
- removed the REF** at (38.0, 160.0)
- removed the REF** at (48.0, 177.0)
- removed RV1: MIN_DENS, Crossley_Footprints:SMD_TRIM_JLC
- removed RV2: MIN_FREQ, Crossley_Footprints:SMD_TRIM_JLC
- removed RV3: CHANGE_RATE, Crossley_Footprints:SMD_TRIM_JLC
- removed RV4: MAX_DENS, Crossley_Footprints:SMD_TRIM_JLC
- removed RV5: MAX_FREQ, Crossley_Footprints:SMD_TRIM_JLC
- removed U0, U1: 74HC245, Package_SO:SO-20_12.8x7.5mm_P1.27mm
- removed U2, U4: MCP6002-xP, Package_SO:SOIC-8_3.9x4.9mm_P1.27mm
- removed U3: L78M05ABDT-TR, Package_TO_SOT_SMD:TO-252-2
- added REF**: Tayda_Slide_SPDT, HammerheadAudio:Tayda_Slide_SPDT, F.Cu at (115.0, 210.0)
- D0, D1, D10, D11, D12, D13, D14, D15, D16, D17, D18, D19, D2, D20, D21, D22, D23, D24, D25, D26, D27, D28, D29, D3, D30, D31, D4, D5, D6, D7, D8, D9: moved to B.Cu
- moved D19 383.8 mm to (30.0, 143.0)
- moved J0 346.2 mm to (50.0, 75.0)
- moved D17 340.0 mm to (60.0, 126.0)
- moved D3 338.4 mm to (70.0, 75.0)
- moved J9 337.2 mm to (30.0, 143.0)
- moved J4 329.8 mm to (30.0, 109.0)
- moved D1 324.0 mm to (50.0, 75.0)
- moved D15 319.5 mm to (40.0, 126.0)
- moved J3 318.5 mm to (60.0, 92.0)
- moved D25 306.5 mm to (40.0, 160.0)
- moved D11 305.2 mm to (50.0, 109.0)
- moved J7 302.9 mm to (40.0, 126.0)
- moved D27 301.5 mm to (60.0, 160.0)
- moved J2 301.2 mm to (40.0, 92.0)
- moved J10 299.8 mm to (50.0, 143.0)
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Routing:
- removed copper zone on F.Cu, net /NET1
Other:
- board outline added: 115.8 x 162.5 mm

Commit message: alterantive sketch
Parts:
- added C1: 0.33uf, Capacitor_SMD:C_0603_1608Metric_Pad1.05x0.95mm_HandSolder_SmallRef, F.Cu at (199.9, 152.2)
- added C2: 0.1uf, Capacitor_SMD:C_0603_1608Metric_Pad1.05x0.95mm_HandSolder_SmallRef, F.Cu at (217.3, 152.9)
- added D32: SM4007PL, Diode_SMD:D_SOD-123, F.Cu at (186.8, 144.7)
- added D33: SM4007PL, Diode_SMD:D_SOD-123, F.Cu at (199.0, 136.6)
- added D34: SM4007PL, Diode_SMD:D_SOD-123, F.Cu at (186.8, 148.0)
- added D35: SM4007PL, Diode_SMD:D_SOD-123, F.Cu at (207.4, 130.2)
- added H3: M3/#4-40, HammerheadAudio:M3_Plated, F.Cu at (26.0, 129.0)
- added H3: M3/#4-40, HammerheadAudio:M3_Plated, F.Cu at (74.0, 89.0)
- added H3: M3/#4-40, HammerheadAudio:M3_Plated, F.Cu at (36.0, 78.0)
- added J16: FM_IN, HammerheadAudio:EuroJack_MonoSW_THT_NOREF_Mask, F.Cu at (110.0, 210.0)
- added Q1: MMBT3904, Package_TO_SOT_SMD:SOT-23, F.Cu at (191.2, 152.0)
- added Q2: MMBT3904, Package_TO_SOT_SMD:SOT-23, F.Cu at (196.9, 146.2)
- added R0: LRV_R, Resistor_SMD:R_0603_1608Metric_Pad1.05x0.95mm_HandSolder_SmallRef, F.Cu at (212.2, 156.9)
- added R1: WSP_R, Resistor_SMD:R_0603_1608Metric_Pad1.05x0.95mm_HandSolder_SmallRef, F.Cu at (223.6, 144.8)
- added R10: WSP_R, Resistor_SMD:R_0603_1608Metric_Pad1.05x0.95mm_HandSolder_SmallRef, F.Cu at (201.9, 141.8)
- added R11: O_R, Resistor_SMD:R_0603_1608Metric_Pad1.05x0.95mm_HandSolder_SmallRef, F.Cu at (209.0, 135.6)
- added R12: LRV_R, Resistor_SMD:R_0603_1608Metric_Pad1.05x0.95mm_HandSolder_SmallRef, F.Cu at (209.0, 138.1)
- added R13: WSP_R, Resistor_SMD:R_0603_1608Metric_Pad1.05x0.95mm_HandSolder_SmallRef, F.Cu at (201.9, 144.3)
- added R14: O_R, Resistor_SMD:R_0603_1608Metric_Pad1.05x0.95mm_HandSolder_SmallRef, F.Cu at (190.5, 156.6)
- added R15: LRV_R, Resistor_SMD:R_0603_1608Metric_Pad1.05x0.95mm_HandSolder_SmallRef, F.Cu at (196.9, 149.7)
- added R16: WSP_R, Resistor_SMD:R_0603_1608Metric_Pad1.05x0.95mm_HandSolder_SmallRef, F.Cu at (217.5, 129.8)
- added R17: O_R, Resistor_SMD:R_0603_1608Metric_Pad1.05x0.95mm_HandSolder_SmallRef, F.Cu at (206.2, 141.8)
- added R18: LRV_R, Resistor_SMD:R_0603_1608Metric_Pad1.05x0.95mm_HandSolder_SmallRef, F.Cu at (213.4, 135.4)
- added R19: WSP_R, Resistor_SMD:R_0603_1608Metric_Pad1.05x0.95mm_HandSolder_SmallRef, F.Cu at (201.3, 146.8)
- added R2: O_R, Resistor_SMD:R_0603_1608Metric_Pad1.05x0.95mm_HandSolder_SmallRef, F.Cu at (217.3, 150.4)
- added R20: O_R, Resistor_SMD:R_0603_1608Metric_Pad1.05x0.95mm_HandSolder_SmallRef, F.Cu at (195.6, 152.2)
- added R21: LRV_R, Resistor_SMD:R_0603_1608Metric_Pad1.05x0.95mm_HandSolder_SmallRef, F.Cu at (213.4, 137.9)
- added R22: WSP_R, Resistor_SMD:R_0603_1608Metric_Pad1.05x0.95mm_HandSolder_SmallRef, F.Cu at (195.6, 154.7)
- added R23: O_R, Resistor_SMD:R_0603_1608Metric_Pad1.05x0.95mm_HandSolder_SmallRef, F.Cu at (201.3, 149.3)
- added R24: LRV_R, Resistor_SMD:R_0603_1608Metric_Pad1.05x0.95mm_HandSolder_SmallRef, F.Cu at (206.2, 144.3)
- added R25: WSP_R, Resistor_SMD:R_0603_1608Metric_Pad1.05x0.95mm_HandSolder_SmallRef, F.Cu at (217.5, 132.3)
- added R26: O_R, Resistor_SMD:R_0603_1608Metric_Pad1.05x0.95mm_HandSolder_SmallRef, F.Cu at (221.8, 129.8)
- added R27: LRV_R, Resistor_SMD:R_0603_1608Metric_Pad1.05x0.95mm_HandSolder_SmallRef, F.Cu at (210.6, 140.6)
- added R28: WSP_R, Resistor_SMD:R_0603_1608Metric_Pad1.05x0.95mm_HandSolder_SmallRef, F.Cu at (223.6, 147.3)
- added R29: O_R, Resistor_SMD:R_0603_1608Metric_Pad1.05x0.95mm_HandSolder_SmallRef, F.Cu at (217.7, 134.8)
- added R3: LRV_R, Resistor_SMD:R_0603_1608Metric_Pad1.05x0.95mm_HandSolder_SmallRef, F.Cu at (213.0, 153.2)
- added R30: LRV_R, Resistor_SMD:R_0603_1608Metric_Pad1.05x0.95mm_HandSolder_SmallRef, F.Cu at (205.7, 146.8)
- added R31: WSP_R, Resistor_SMD:R_0603_1608Metric_Pad1.05x0.95mm_HandSolder_SmallRef, F.Cu at (194.8, 157.2)
- added R32: O_R, Resistor_SMD:R_0603_1608Metric_Pad1.05x0.95mm_HandSolder_SmallRef, F.Cu at (210.6, 143.1)
- added R33: LRV_R, Resistor_SMD:R_0603_1608Metric_Pad1.05x0.95mm_HandSolder_SmallRef, F.Cu at (217.7, 137.3)
- added R34: WSP_R, Resistor_SMD:R_0603_1608Metric_Pad1.05x0.95mm_HandSolder_SmallRef, F.Cu at (205.7, 149.3)
- added R35: O_R, Resistor_SMD:R_0603_1608Metric_Pad1.05x0.95mm_HandSolder_SmallRef, F.Cu at (199.9, 154.7)
- added R36: LRV_R, Resistor_SMD:R_0603_1608Metric_Pad1.05x0.95mm_HandSolder_SmallRef, F.Cu at (214.9, 140.4)
- added R37: WSP_R, Resistor_SMD:R_0603_1608Metric_Pad1.05x0.95mm_HandSolder_SmallRef, F.Cu at (221.8, 132.3)
- added R38: O_R, Resistor_SMD:R_0603_1608Metric_Pad1.05x0.95mm_HandSolder_SmallRef, F.Cu at (204.3, 151.8)
- added R39: LRV_R, Resistor_SMD:R_0603_1608Metric_Pad1.05x0.95mm_HandSolder_SmallRef, F.Cu at (210.6, 145.7)
- added R4: WSP_R, Resistor_SMD:R_0603_1608Metric_Pad1.05x0.95mm_HandSolder_SmallRef, F.Cu at (219.3, 147.3)
- added R40: WSP_R, Resistor_SMD:R_0603_1608Metric_Pad1.05x0.95mm_HandSolder_SmallRef, F.Cu at (199.2, 157.2)
- added R41: O_R, Resistor_SMD:R_0603_1608Metric_Pad1.05x0.95mm_HandSolder_SmallRef, F.Cu at (222.1, 134.8)
- added R42: LRV_R, Resistor_SMD:R_0603_1608Metric_Pad1.05x0.95mm_HandSolder_SmallRef, F.Cu at (214.9, 142.9)
- added R43: WSP_R, Resistor_SMD:R_0603_1608Metric_Pad1.05x0.95mm_HandSolder_SmallRef, F.Cu at (222.1, 137.3)
- added R44: O_R, Resistor_SMD:R_0603_1608Metric_Pad1.05x0.95mm_HandSolder_SmallRef, F.Cu at (210.0, 148.2)
- added R45: LRV_R, Resistor_SMD:R_0603_1608Metric_Pad1.05x0.95mm_HandSolder_SmallRef, F.Cu at (204.3, 154.4)
- added R46: WSP_R, Resistor_SMD:R_0603_1608Metric_Pad1.05x0.95mm_HandSolder_SmallRef, F.Cu at (219.3, 139.8)
- added R47: O_R, Resistor_SMD:R_0603_1608Metric_Pad1.05x0.95mm_HandSolder_SmallRef, F.Cu at (208.6, 151.8)
- added R48: 100k, Resistor_SMD:R_0603_1608Metric_Pad1.05x0.95mm_HandSolder_SmallRef, F.Cu at (214.9, 145.4)
- added R49: 100k, Resistor_SMD:R_0603_1608Metric_Pad1.05x0.95mm_HandSolder_SmallRef, F.Cu at (203.5, 157.2)
- added R5: O_R, Resistor_SMD:R_0603_1608Metric_Pad1.05x0.95mm_HandSolder_SmallRef, F.Cu at (223.6, 142.3)
- added R50: 1k, Resistor_SMD:R_0603_1608Metric_Pad1.05x0.95mm_HandSolder_SmallRef, F.Cu at (219.3, 142.3)
- added R51: 100k, Resistor_SMD:R_0603_1608Metric_Pad1.05x0.95mm_HandSolder_SmallRef, F.Cu at (214.9, 147.9)
- added R52: 100k, Resistor_SMD:R_0603_1608Metric_Pad1.05x0.95mm_HandSolder_SmallRef, F.Cu at (208.6, 154.4)
- added R53: 100k, Resistor_SMD:R_0603_1608Metric_Pad1.05x0.95mm_HandSolder_SmallRef, F.Cu at (223.6, 139.8)
- added R54: 100k, Resistor_SMD:R_0603_1608Metric_Pad1.05x0.95mm_HandSolder_SmallRef, F.Cu at (213.0, 150.7)
- added R6: LRV_R, Resistor_SMD:R_0603_1608Metric_Pad1.05x0.95mm_HandSolder_SmallRef, F.Cu at (207.9, 156.9)
- added R7: WSP_R, Resistor_SMD:R_0603_1608Metric_Pad1.05x0.95mm_HandSolder_SmallRef, F.Cu at (219.3, 144.8)
- added R8: O_R, Resistor_SMD:R_0603_1608Metric_Pad1.05x0.95mm_HandSolder_SmallRef, F.Cu at (206.7, 133.1)
- added R9: LRV_R, Resistor_SMD:R_0603_1608Metric_Pad1.05x0.95mm_HandSolder_SmallRef, F.Cu at (186.1, 156.6)
- added RV1: MIN_DENS, Crossley_Footprints:SMD_TRIM_JLC, F.Cu at (80.0, 185.0)
- added RV2: MIN_FREQ, Crossley_Footprints:SMD_TRIM_JLC, F.Cu at (95.0, 185.0)
- added RV3: CHANGE_RATE, Crossley_Footprints:SMD_TRIM_JLC, F.Cu at (110.0, 185.0)
- added RV4: MAX_DENS, Crossley_Footprints:SMD_TRIM_JLC, F.Cu at (80.0, 195.0)
- added RV5: MAX_FREQ, Crossley_Footprints:SMD_TRIM_JLC, F.Cu at (95.0, 195.0)
- added U0: 74HC245, Package_SO:SO-20_12.8x7.5mm_P1.27mm, F.Cu at (177.7, 150.2)
- added U1: 74HC245, Package_SO:SO-20_12.8x7.5mm_P1.27mm, F.Cu at (177.7, 135.7)
- added U2: MCP6002-xP, Package_SO:SOIC-8_3.9x4.9mm_P1.27mm, F.Cu at (188.2, 139.8)
- added U3: L78M05ABDT-TR, Package_TO_SOT_SMD:TO-252-2, F.Cu at (190.0, 132.5)
- added U4: MCP6002-xP, Package_SO:SOIC-8_3.9x4.9mm_P1.27mm, F.Cu at (200.3, 131.7)
- U5: footprint MeowWolf_Templates:TEENSY_LC_NO_SILK -> MeowWolf_Templates:TEENSY_LC_MIN_SILK_2SIDE
- moved D19 52.8 mm to (80.0, 126.0)
- moved J9 52.8 mm to (80.0, 126.0)
- moved D25 34.5 mm to (70.0, 143.0)
- moved J12 34.5 mm to (70.0, 143.0)
- moved D21 20.0 mm to (30.0, 143.0)
- moved D23 20.0 mm to (50.0, 143.0)
- moved D27 20.0 mm to (40.0, 160.0)
- moved D29 20.0 mm to (60.0, 160.0)
- moved J10 20.0 mm to (30.0, 143.0)
- moved J11 20.0 mm to (50.0, 143.0)
- moved J13 20.0 mm to (40.0, 160.0)
- moved J14 20.0 mm to (60.0, 160.0)
- moved U5 14.1 mm to (125.0, 165.0)
- moved G*** 13.5 mm to (125.0, 166.0) (x2)
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Routing:
- added copper zone on B.Cu, net /NET2
- added copper zone on B.Cu, net GND
Other:
- board size 115.8 x 162.5 mm -> 125.8 x 167.5 mm

Commit message: Finished schematic
Parts:
- removed C1: 0.33uf, Capacitor_SMD:C_0603_1608Metric_Pad1.05x0.95mm_HandSolder_SmallRef
- removed C2: 0.1uf, Capacitor_SMD:C_0603_1608Metric_Pad1.05x0.95mm_HandSolder_SmallRef
- removed D32, D33, D34, D35: SM4007PL, Diode_SMD:D_SOD-123
- removed Q1, Q2: MMBT3904, Package_TO_SOT_SMD:SOT-23
- removed R0, R12, R15, R18, R21, R24, R27, R3, R30, R33, R36, R39, R42, R45, R6, R9: LRV_R, Resistor_SMD:R_0603_1608Metric_Pad1.05x0.95mm_HandSolder_SmallRef
- removed R1, R10, R13, R16, R19, R22, R25, R28, R31, R34, R37, R4, R40, R43, R46, R7: WSP_R, Resistor_SMD:R_0603_1608Metric_Pad1.05x0.95mm_HandSolder_SmallRef
- removed R11, R14, R17, R2, R20, R23, R26, R29, R32, R35, R38, R41, R44, R47, R5, R8: O_R, Resistor_SMD:R_0603_1608Metric_Pad1.05x0.95mm_HandSolder_SmallRef
- removed R48, R49, R51, R52, R53, R54: 100k, Resistor_SMD:R_0603_1608Metric_Pad1.05x0.95mm_HandSolder_SmallRef
- removed R50: 1k, Resistor_SMD:R_0603_1608Metric_Pad1.05x0.95mm_HandSolder_SmallRef
- removed U0, U1: 74HC245, Package_SO:SO-20_12.8x7.5mm_P1.27mm
- removed U2, U4: MCP6002-xP, Package_SO:SOIC-8_3.9x4.9mm_P1.27mm
- removed U3: L78M05ABDT-TR, Package_TO_SOT_SMD:TO-252-2

Commit message: layout ideas
Parts:
- removed H3 (x6): M3/#4-40, HammerheadAudio:M3_Plated
- removed the J16 at (110.0, 210.0)
- removed REF**: Tayda_Slide_SPDT, HammerheadAudio:Tayda_Slide_SPDT
- removed RV5: MAX_FREQ, Crossley_Footprints:SMD_TRIM_JLC
- added C1: 0.33uf, Capacitor_SMD:C_0603_1608Metric_Pad1.05x0.95mm_HandSolder_SmallRef_Fab, F.Cu at (123.2, 197.8)
- added C2: 0.1uf, Capacitor_SMD:C_0603_1608Metric_Pad1.05x0.95mm_HandSolder_SmallRef_Fab, F.Cu at (107.8, 146.2)
- added C3: 0.1uf, Capacitor_SMD:C_0603_1608Metric_Pad1.05x0.95mm_HandSolder_SmallRef_Fab, F.Cu at (123.5, 177.2)
- added C4: 0.1uf, Capacitor_SMD:C_0603_1608Metric_Pad1.05x0.95mm_HandSolder_SmallRef_Fab, F.Cu at (122.8, 167.8)
- added C5: 0.1uf, Capacitor_SMD:C_0603_1608Metric_Pad1.05x0.95mm_HandSolder_SmallRef_Fab, F.Cu at (107.8, 130.5)
- added C6: 0.1uf, Capacitor_SMD:C_0603_1608Metric_Pad1.05x0.95mm_HandSolder_SmallRef_Fab, F.Cu at (126.8, 197.8)
- added D32: DENS1, LED_SMD:LED_1206_3216Metric_Pad1.42x1.75mm_HandSolder_FabRef, B.Cu at (121.5, 141.5)
- added D33: SM4007PL, Diode_SMD:D_SOD-123, F.Cu at (129.2, 173.8)
- added D34: DROP, LED_SMD:LED_1206_3216Metric_Pad1.42x1.75mm_HandSolder_FabRef, B.Cu at (121.5, 156.0)
- added D35: SM4007PL, Diode_SMD:D_SOD-123, F.Cu at (129.2, 168.8)
- added D36: SM4007PL, Diode_SMD:D_SOD-123, F.Cu at (118.0, 198.0)
- added D37: PANIC, LED_SMD:LED_1206_3216Metric_Pad1.42x1.75mm_HandSolder_FabRef, B.Cu at (65.0, 210.0)
- added D38: M7, Diode_SMD:D_SMA, F.Cu at (125.0, 200.5)
- added D39: DENS2, LED_SMD:LED_1206_3216Metric_Pad1.42x1.75mm_HandSolder_FabRef, B.Cu at (80.0, 210.0)
- added D40: DENS3, LED_SMD:LED_1206_3216Metric_Pad1.42x1.75mm_HandSolder_FabRef, B.Cu at (95.0, 210.0)
- added D41: DROP2, LED_SMD:LED_1206_3216Metric_Pad1.42x1.75mm_HandSolder_FabRef, B.Cu at (110.0, 210.0)
- added G***: LOGO, Skelly:Hand1_Smooth_2.9x5.8mm, F.Cu at (120.0, 207.0)
- added G***: LOGO, Skelly:Hand1_Smooth_2.9x5.8mm, F.Cu at (120.0, 213.0)
- added G***: LOGO, HammerheadAudio:Hand_Open_5x5.5mm_Silk, F.Cu at (80.0, 199.0)
- added G***: LOGO, HammerheadAudio:Hand_Open_5x5.5mm_Silk, F.Cu at (95.0, 199.0)
- added G***: LOGO, HammerheadAudio:BeeHive_Icon_6.3x5.8mm, F.Cu at (87.5, 199.0)
- added G***: LOGO, Skelly:Hand1_Smooth_2.9x5.8mm_Back, B.Cu at (130.0, 213.0)
- added G***: LOGO, Skelly:Hand1_Smooth_2.9x5.8mm_Back, B.Cu at (130.0, 207.0)
- added G***: LOGO, HammerheadAudio:Panic2_5.8x5.8mm, F.Cu at (65.0, 199.0)
- added G***: LOGO, HammerheadAudio:HoneyDrop_Icon_4x5.8mm, F.Cu at (110.0, 199.0)
- added J19: PANIC_IN, HammerheadAudio:EuroJack_MonoSW_THT_NOREF_Mask, F.Cu at (65.0, 210.0)
- added J20: GND, HammerheadAudio:M3_Plated, F.Cu at (74.0, 89.0)
- added J21: GND, HammerheadAudio:M3_Plated, F.Cu at (50.0, 225.0)
- added J22: GND, HammerheadAudio:M3_Plated, F.Cu at (36.0, 78.0)
- added J23: GND, HammerheadAudio:M3_Plated, F.Cu at (140.0, 120.0)
- added J24: GND, HammerheadAudio:M3_Plated, F.Cu at (26.0, 129.0)
- added J25: PWR, HammerheadAudio:M3_Plated, F.Cu at (140.0, 225.0)
- added Q1: MMBT3904, Package_TO_SOT_SMD:SOT-23, F.Cu at (117.8, 188.0)
- added Q2: MMBT3904, Package_TO_SOT_SMD:SOT-23, F.Cu at (117.8, 193.5)
- added R0: LRV_R, Resistor_SMD:R_0603_1608Metric_Pad1.05x0.95mm_HandSolder_SmallRef_Fab, F.Cu at (95.0, 125.0)
- added R1: WSP_R, Resistor_SMD:R_0603_1608Metric_Pad1.05x0.95mm_HandSolder_SmallRef_Fab, F.Cu at (56.0, 77.0)
- added R10: WSP_R, Resistor_SMD:R_0603_1608Metric_Pad1.05x0.95mm_HandSolder_SmallRef_Fab, F.Cu at (66.0, 94.0)
- added R11: O_R, Resistor_SMD:R_0603_1608Metric_Pad1.05x0.95mm_HandSolder_SmallRef_Fab, F.Cu at (66.0, 90.0)
- added R12: LRV_R, Resistor_SMD:R_0603_1608Metric_Pad1.05x0.95mm_HandSolder_SmallRef_Fab, F.Cu at (135.0, 150.0)
- added R13: WSP_R, Resistor_SMD:R_0603_1608Metric_Pad1.05x0.95mm_HandSolder_SmallRef_Fab, F.Cu at (36.0, 111.0)
- added R14: O_R, Resistor_SMD:R_0603_1608Metric_Pad1.05x0.95mm_HandSolder_SmallRef_Fab, F.Cu at (36.0, 107.0)
- added R15: LRV_R, Resistor_SMD:R_0603_1608Metric_Pad1.05x0.95mm_HandSolder_SmallRef_Fab, F.Cu at (135.0, 165.0)
- added R16: WSP_R, Resistor_SMD:R_0603_1608Metric_Pad1.05x0.95mm_HandSolder_SmallRef_Fab, F.Cu at (56.0, 111.0)
- added R17: O_R, Resistor_SMD:R_0603_1608Metric_Pad1.05x0.95mm_HandSolder_SmallRef_Fab, F.Cu at (56.0, 107.0)
- added R18: LRV_R, Resistor_SMD:R_0603_1608Metric_Pad1.05x0.95mm_HandSolder_SmallRef_Fab, F.Cu at (135.0, 180.0)
- added R19: WSP_R, Resistor_SMD:R_0603_1608Metric_Pad1.05x0.95mm_HandSolder_SmallRef_Fab, F.Cu at (76.0, 111.0)
- added R2: O_R, Resistor_SMD:R_0603_1608Metric_Pad1.05x0.95mm_HandSolder_SmallRef_Fab, F.Cu at (56.0, 73.0)
- added R20: O_R, Resistor_SMD:R_0603_1608Metric_Pad1.05x0.95mm_HandSolder_SmallRef_Fab, F.Cu at (76.0, 107.0)
- added R21: LRV_R, Resistor_SMD:R_0603_1608Metric_Pad1.05x0.95mm_HandSolder_SmallRef_Fab, F.Cu at (135.0, 195.0)
- added R22: WSP_R, Resistor_SMD:R_0603_1608Metric_Pad1.05x0.95mm_HandSolder_SmallRef_Fab, F.Cu at (46.0, 128.0)
- added R23: O_R, Resistor_SMD:R_0603_1608Metric_Pad1.05x0.95mm_HandSolder_SmallRef_Fab, F.Cu at (46.0, 124.0)
- added R24: LRV_R, Resistor_SMD:R_0603_1608Metric_Pad1.05x0.95mm_HandSolder_SmallRef_Fab, F.Cu at (135.0, 210.0)
- added R25: WSP_R, Resistor_SMD:R_0603_1608Metric_Pad1.05x0.95mm_HandSolder_SmallRef_Fab, F.Cu at (66.0, 128.0)
- added R26: O_R, Resistor_SMD:R_0603_1608Metric_Pad1.05x0.95mm_HandSolder_SmallRef_Fab, F.Cu at (66.0, 124.0)
- added R27: LRV_R, Resistor_SMD:R_0603_1608Metric_Pad1.05x0.95mm_HandSolder_SmallRef_Fab, F.Cu at (125.0, 220.0)
- added R28: WSP_R, Resistor_SMD:R_0603_1608Metric_Pad1.05x0.95mm_HandSolder_SmallRef_Fab, F.Cu at (86.0, 128.0)
- added R29: O_R, Resistor_SMD:R_0603_1608Metric_Pad1.05x0.95mm_HandSolder_SmallRef_Fab, F.Cu at (86.0, 124.0)
- added R3: LRV_R, Resistor_SMD:R_0603_1608Metric_Pad1.05x0.95mm_HandSolder_SmallRef_Fab, F.Cu at (110.0, 125.0)
- added R30: LRV_R, Resistor_SMD:R_0603_1608Metric_Pad1.05x0.95mm_HandSolder_SmallRef_Fab, F.Cu at (110.0, 220.0)
- added R31: WSP_R, Resistor_SMD:R_0603_1608Metric_Pad1.05x0.95mm_HandSolder_SmallRef_Fab, F.Cu at (36.0, 145.0)
- added R32: O_R, Resistor_SMD:R_0603_1608Metric_Pad1.05x0.95mm_HandSolder_SmallRef_Fab, F.Cu at (36.0, 141.0)
- added R33: LRV_R, Resistor_SMD:R_0603_1608Metric_Pad1.05x0.95mm_HandSolder_SmallRef_Fab, F.Cu at (95.0, 220.0)
- added R34: WSP_R, Resistor_SMD:R_0603_1608Metric_Pad1.05x0.95mm_HandSolder_SmallRef_Fab, F.Cu at (56.0, 145.1)
- added R35: O_R, Resistor_SMD:R_0603_1608Metric_Pad1.05x0.95mm_HandSolder_SmallRef_Fab, F.Cu at (56.0, 141.0)
- added R36: LRV_R, Resistor_SMD:R_0603_1608Metric_Pad1.05x0.95mm_HandSolder_SmallRef_Fab, F.Cu at (80.0, 220.0)
- added R37: WSP_R, Resistor_SMD:R_0603_1608Metric_Pad1.05x0.95mm_HandSolder_SmallRef_Fab, F.Cu at (76.0, 145.0)
- added R38: O_R, Resistor_SMD:R_0603_1608Metric_Pad1.05x0.95mm_HandSolder_SmallRef_Fab, F.Cu at (76.0, 141.0)
- added R39: LRV_R, Resistor_SMD:R_0603_1608Metric_Pad1.05x0.95mm_HandSolder_SmallRef_Fab, F.Cu at (65.0, 220.0)
- added R4: WSP_R, Resistor_SMD:R_0603_1608Metric_Pad1.05x0.95mm_HandSolder_SmallRef_Fab, F.Cu at (76.0, 77.0)
- added R40: WSP_R, Resistor_SMD:R_0603_1608Metric_Pad1.05x0.95mm_HandSolder_SmallRef_Fab, F.Cu at (46.0, 162.0)
- added R41: O_R, Resistor_SMD:R_0603_1608Metric_Pad1.05x0.95mm_HandSolder_SmallRef_Fab, F.Cu at (46.0, 158.0)
- added R42: LRV_R, Resistor_SMD:R_0603_1608Metric_Pad1.05x0.95mm_HandSolder_SmallRef_Fab, F.Cu at (55.0, 210.0)
- added R43: WSP_R, Resistor_SMD:R_0603_1608Metric_Pad1.05x0.95mm_HandSolder_SmallRef_Fab, F.Cu at (66.0, 162.0)
- added R44: O_R, Resistor_SMD:R_0603_1608Metric_Pad1.05x0.95mm_HandSolder_SmallRef_Fab, F.Cu at (66.0, 158.0)
- added R45: LRV_R, Resistor_SMD:R_0603_1608Metric_Pad1.05x0.95mm_HandSolder_SmallRef_Fab, F.Cu at (55.0, 195.0)
- added R46: WSP_R, Resistor_SMD:R_0603_1608Metric_Pad1.05x0.95mm_HandSolder_SmallRef_Fab, F.Cu at (56.0, 179.0)
- added R47: O_R, Resistor_SMD:R_0603_1608Metric_Pad1.05x0.95mm_HandSolder_SmallRef_Fab, F.Cu at (56.0, 175.0)
- added R48: 1k, Resistor_SMD:R_0603_1608Metric_Pad1.05x0.95mm_HandSolder_SmallRef_Fab, F.Cu at (119.5, 177.2)
- added R49: 100k, Resistor_SMD:R_0603_1608Metric_Pad1.05x0.95mm_HandSolder_SmallRef_Fab, F.Cu at (129.5, 182.0)
- added R5: O_R, Resistor_SMD:R_0603_1608Metric_Pad1.05x0.95mm_HandSolder_SmallRef_Fab, F.Cu at (76.0, 73.0)
- added R50: 100k, Resistor_SMD:R_0603_1608Metric_Pad1.05x0.95mm_HandSolder_SmallRef_Fab, F.Cu at (126.5, 182.0)
- added R51: 100k, Resistor_SMD:R_0603_1608Metric_Pad1.05x0.95mm_HandSolder_SmallRef_Fab, F.Cu at (126.5, 173.8)
- added R52: 100k, Resistor_SMD:R_0603_1608Metric_Pad1.05x0.95mm_HandSolder_SmallRef_Fab, F.Cu at (115.5, 182.0)
- added R53: 100k, Resistor_SMD:R_0603_1608Metric_Pad1.05x0.95mm_HandSolder_SmallRef_Fab, F.Cu at (126.5, 168.8)
- added R54: 100k, Resistor_SMD:R_0603_1608Metric_Pad1.05x0.95mm_HandSolder_SmallRef_Fab, F.Cu at (115.5, 178.2)
- added R55: 1k, Resistor_SMD:R_0603_1608Metric_Pad1.05x0.95mm_HandSolder_SmallRef_Fab, F.Cu at (129.5, 178.2)
- added R56: 100k, Resistor_SMD:R_0603_1608Metric_Pad1.05x0.95mm_HandSolder_SmallRef_Fab, F.Cu at (113.2, 178.2)
- added R57: 47k, Resistor_SMD:R_0603_1608Metric_Pad1.05x0.95mm_HandSolder_SmallRef_Fab, F.Cu at (115.5, 173.8)
- added R58: DENS_R, Resistor_SMD:R_0603_1608Metric_Pad1.05x0.95mm_HandSolder_SmallRef_Fab, F.Cu at (126.5, 178.2)
- added R59: WSP_R, Resistor_SMD:R_0603_1608Metric_Pad1.05x0.95mm_HandSolder_SmallRef_Fab, F.Cu at (115.5, 168.8)
- added R6: LRV_R, Resistor_SMD:R_0603_1608Metric_Pad1.05x0.95mm_HandSolder_SmallRef_Fab, F.Cu at (125.0, 125.0)
- added R60: 1k, Resistor_SMD:R_0603_1608Metric_Pad1.05x0.95mm_HandSolder_SmallRef_Fab, F.Cu at (117.8, 200.0)
- added R61: 100k, Resistor_SMD:R_0603_1608Metric_Pad1.05x0.95mm_HandSolder_SmallRef_Fab, F.Cu at (117.8, 196.0)
- added R62: GP_R, Resistor_SMD:R_0603_1608Metric_Pad1.05x0.95mm_HandSolder_SmallRef_Fab, F.Cu at (71.0, 210.0)
- added R63: 1k, Resistor_SMD:R_0603_1608Metric_Pad1.05x0.95mm_HandSolder_SmallRef_Fab, F.Cu at (117.8, 190.8)
- added R64: DENS_R, Resistor_SMD:R_0603_1608Metric_Pad1.05x0.95mm_HandSolder_SmallRef_Fab, F.Cu at (86.0, 210.0)
- added R65: DENS_R, Resistor_SMD:R_0603_1608Metric_Pad1.05x0.95mm_HandSolder_SmallRef_Fab, F.Cu at (101.0, 210.0)
- added R66: WSP_R, Resistor_SMD:R_0603_1608Metric_Pad1.05x0.95mm_HandSolder_SmallRef_Fab, F.Cu at (116.0, 210.0)
- added R67: 1k, Resistor_SMD:R_0603_1608Metric_Pad1.05x0.95mm_HandSolder_SmallRef_Fab, F.Cu at (113.2, 173.8)
- added R7: WSP_R, Resistor_SMD:R_0603_1608Metric_Pad1.05x0.95mm_HandSolder_SmallRef_Fab, F.Cu at (46.0, 94.0)
- added R8: O_R, Resistor_SMD:R_0603_1608Metric_Pad1.05x0.95mm_HandSolder_SmallRef_Fab, F.Cu at (46.0, 90.0)
- added R9: LRV_R, Resistor_SMD:R_0603_1608Metric_Pad1.05x0.95mm_HandSolder_SmallRef_Fab, F.Cu at (135.0, 135.0)
- added SW1: SW_SPDT, HammerheadAudio:Tayda_Slide_SPDT, F.Cu at (125.0, 210.0)
- added U0: 74HC245, Package_SO:SOIC-20W_7.5x12.8mm_P1.27mm, F.Cu at (104.0, 138.2)
- added U1: 74HC245, Package_SO:SOIC-20W_7.5x12.8mm_P1.27mm, F.Cu at (104.0, 153.8)
- added U2: MCP6002-xP, Package_SO:SOIC-8_3.9x4.9mm_P1.27mm, F.Cu at (120.8, 172.0)
- added U3: MCP6002-xP, Package_SO:SOIC-8_3.9x4.9mm_P1.27mm, F.Cu at (121.5, 181.0)
- added U4: TEENSY_3.2_MINIMAL, MeowWolf_Templates:TEENSY_LC_MIN_SILK_2SIDE, B.Cu at (121.5, 147.5)
- D1, D11, D13, D15, D17, D19, D21, D23, D25, D27, D29, D3, D31, D5, D7, D9: footprint LED_SMD:LED_1206_3216Metric_Pad1.42x1.75mm_HandSolder -> LED_SMD:LED_1206_3216Metric_Pad1.42x1.75mm_HandSolder_FabRef
- J16: value FM_IN -> DENS_OUT
- J18: value DENS_IN -> DROP_OUT
- RV2: value MIN_FREQ -> MAX_DENS
- RV4: value MAX_DENS -> XCTRL
- U5: value TEENSY_3.2_MINIMAL -> L78M05ABDT-TR; footprint MeowWolf_Templates:TEENSY_LC_MIN_SILK_2SIDE -> Package_TO_SOT_SMD:TO-252-2; moved to F.Cu
- moved J18 45.0 mm to (110.0, 210.0)
- moved RV4 30.5 mm to (110.0, 189.8)
- moved U5 26.2 mm to (125.0, 191.2), turned to 90 degrees
- moved G*** 17.8 mm to (121.5, 148.5) (x3)
- moved RV1 15.7 mm to (65.0, 189.8)
- moved RV2 15.7 mm to (80.0, 189.8)
- moved RV3 15.7 mm to (95.0, 189.8)
Connections:
- J16 pad 1: /FM_IN -> Net-(J16-Pad1)
- J17 pad 3: /DENS_NORM -> Net-(J17-Pad3)
- J18 pad 1: (no net) -> Net-(J18-Pad1)
- J18 pad 2: (no net) -> GND
- RV1 pad 2: (no net) -> MIN_DENS
- RV2 pad 2: (no net) -> MAX_DENS
- RV3 pad 2: (no net) -> ROC
- RV4 pad 2: (no net) -> XCTRL
- U5 pad 1: (no net) -> VDD
- U5 pad 2: (no net) -> GND
- U5 pad 3: (no net) -> +5V
Routing:
- added copper zone on F.Cu, net GND

Commit message: layout progress
Parts:
- removed the G*** at (80.0, 199.0)
- removed the G*** at (95.0, 199.0)
- added G***: LOGO, HammerheadAudio:Candle_Smooth_2x5.8mm, F.Cu at (128.0, 172.0)
- added G***: LOGO, HammerheadAudio:Globus_Icon_4x5.8mm_Silk, F.Cu at (121.5, 136.0)
- added G***: LOGO, HammerheadAudio:Hand_Open_5x5.5mm_Silk, F.Cu at (108.0, 172.2)
- added G***: LOGO, HammerheadAudio:Hand_Open_5x5.5mm_Silk, F.Cu at (118.0, 172.0)
- added G***: LOGO, Skelly:Hourglass_Smooth_3.3x5.8mm, F.Cu at (98.0, 172.0)
- added G***: LOGO, HammerheadAudio:Globus_Icon_4x5.8mm_Silk, F.Cu at (95.0, 199.0)
- moved D35 53.1 mm to (80.0, 188.5), turned to 0 degrees
- moved D33 50.8 mm to (80.0, 186.0), turned to 180 degrees
- moved R53 46.3 mm to (83.8, 186.5)
- moved R51 45.8 mm to (83.8, 190.2)
- moved R60 44.6 mm to (74.2, 190.2), turned to 90 degrees
- moved Q2 43.1 mm to (75.2, 186.5), turned to 0 degrees
- moved R61 41.9 mm to (76.2, 190.2), turned to 270 degrees
- moved C4 41.5 mm to (85.8, 186.5), turned to 90 degrees
- moved D36 38.6 mm to (80.0, 191.0)
- moved R64 37.9 mm to (115.8, 186.5)
- moved RV1 34.7 mm to (98.0, 179.0)
- moved U2 34.6 mm to (90.8, 189.2)
- moved RV2 30.0 mm to (108.0, 179.0)
- moved R66 29.8 mm to (97.8, 186.5)
- moved R59 29.2 mm to (95.8, 190.2)
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Connections:
- C4 pad 1: +3V3 -> +5V
- U2 pad 1: Net-(R57-Pad1) -> DENS_CV
- U2 pad 2: Net-(R56-Pad2) -> DENS_CV
- U2 pad 3: DROP -> Net-(D33-Pad1)
- U2 pad 5: Net-(D33-Pad1) -> DROP
- U2 pad 6: DENS_CV -> Net-(R56-Pad2)
- U2 pad 7: DENS_CV -> Net-(R57-Pad1)
- U2 pad 8: +3V3 -> +5V

Commit message: layout
Parts:
- moved R64 5.48 mm to (111.8, 190.2), turned to 90 degrees
- moved Q1 4.25 mm to (114.8, 186.5), turned to 0 degrees
- moved R58 4.25 mm to (115.8, 190.2), turned to 90 degrees
- moved R49 3.75 mm to (109.8, 186.5), turned to 270 degrees
- moved R50 3.75 mm to (109.8, 190.2), turned to 90 degrees
- moved R65 2.00 mm to (113.8, 190.2)
- moved D38 0.50 mm to (125.0, 200.2)
- moved C1 0.25 mm to (123.2, 197.2)
- moved C6 0.25 mm to (126.8, 197.2)
