File: Wasp_Hive.kicad_pcb (KiCad board)
At the start: 2 copper layers, 125.8 x 167.5 mm, 171 parts, among them J0 WASP_OUT, J1 WASP_OUT, J10 WASP_OUT, J11 WASP_OUT, J12 WASP_OUT, J13 WASP_OUT, J14 WASP_OUT, J15 WASP_OUT, J16 DENS_OUT, J17 DENS_IN, J18 DROP_OUT, J19 PANIC_IN, J2 WASP_OUT, J20 GND, J21 GND, J22 GND, J23 GND, J24 GND, J25 PWR, J3 WASP_OUT, J4 WASP_OUT, J5 WASP_OUT, J6 WASP_OUT, J7 WASP_OUT, J8 WASP_OUT, J9 WASP_OUT, Q1 MMBT3904, Q2 MMBT3904, SW1 SW_SPDT, U0 74HC245, U1 74HC245, U2 MCP6002-xP, U3 MCP6002-xP, U4 TEENSY_3.2_MINIMAL, U5 L78M05ABDT-TR

Commit message: alt layout
Parts:
- moved G*** 60.0 mm to (70.0, 207.0)
- moved G*** 60.0 mm to (60.0, 213.0)
- moved G*** 60.0 mm to (70.0, 213.0)
- moved G*** 60.0 mm to (60.0, 207.0)
- moved SW1 60.0 mm to (65.0, 210.0)
- moved RV1 31.1 mm to (122.2, 159.5)
- moved G*** 30.4 mm to (122.2, 153.8)
- moved U4 23.5 mm to (110.0, 168.0)
- moved D32 23.5 mm to (110.0, 163.8)
- moved D34 23.5 mm to (110.0, 179.2)
- moved G*** 23.5 mm to (110.0, 171.5) (x3)
- moved G*** 23.5 mm to (110.0, 156.5)
- moved C2 21.8 mm to (98.0, 167.8)
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
Commit message: commit before trying shit
Parts:
- added G***: LOGO, HammerheadAudio:Asterism_5.6x5.5mm_Silk, F.Cu at (65.0, 199.5)
- added R61: 100k, Resistor_SMD:R_0603_1608Metric_Pad1.05x0.95mm_HandSolder_SmallRef_Fab, F.Cu at (102.0, 188.0)
- moved D38 36.5 mm to (91.2, 191.8), turned to 180 degrees
- moved U5 32.0 mm to (93.2, 186.0), turned to 180 degrees
- moved C1 31.6 mm to (99.8, 187.8), turned to 90 degrees
- moved R53 25.4 mm to (121.5, 192.0)
- moved C4 22.6 mm to (121.5, 188.2)
- moved C6 21.9 mm to (99.8, 184.2)
- moved R50 17.9 mm to (131.2, 179.8)
- moved R55 17.9 mm to (129.2, 179.8)
- moved R48 17.0 mm to (123.5, 192.0)
- moved R52 17.0 mm to (130.5, 187.2)
- moved R54 17.0 mm to (126.5, 187.2)
- moved R66 17.0 mm to (123.5, 188.2)
- moved U3 17.0 mm to (128.5, 191.0)
- moved D33 15.0 mm to (105.8, 192.5)
- moved D35 15.0 mm to (105.8, 190.0), turned to 180 degrees
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
Commit message: slightly higher
Parts:
- moved C1 3.50 mm to (99.8, 184.2)
- moved C2 3.50 mm to (97.5, 163.8)
- moved C3 3.50 mm to (125.2, 176.2)
- moved C4 3.50 mm to (121.5, 184.8)
- moved C5 3.50 mm to (97.5, 148.0)
- moved C6 3.50 mm to (99.8, 180.8)
- moved D32 3.50 mm to (110.0, 160.2)
- moved D33 3.50 mm to (105.8, 189.0)
- moved D34 3.50 mm to (110.0, 175.8)
- moved D35 3.50 mm to (105.8, 186.5)
- moved D36 3.50 mm to (105.8, 184.0)
- moved D38 3.50 mm to (91.2, 188.2)
- moved G*** 3.50 mm to (110.0, 168.0) (x3)
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
Commit message: breaking for night
Parts:
- removed the G*** at (65.0, 199.5)
- removed the R61 at (102.0, 184.5)
- moved D38 28.4 mm to (65.0, 199.0)
- moved R64 15.9 mm to (130.8, 190.2), turned to 0 degrees
- moved R55 15.4 mm to (122.8, 190.2), turned to 180 degrees
- moved G*** 12.8 mm to (129.0, 175.0)
- moved R62 12.7 mm to (97.2, 188.2), turned to 0 degrees
- moved R54 12.6 mm to (114.8, 188.2)
- moved C1 12.1 mm to (89.2, 190.2), turned to 0 degrees
- moved R49 12.0 mm to (126.8, 188.2), turned to 180 degrees
- moved C6 11.7 mm to (93.0, 190.2), turned to 180 degrees
- moved C4 11.0 mm to (110.8, 182.2), turned to 180 degrees
- moved R50 11.0 mm to (126.8, 186.2), turned to 0 degrees
- moved R67 10.3 mm to (110.8, 190.2), turned to 0 degrees
- moved R48 9.03 mm to (114.8, 186.2), turned to 0 degrees
- moved RV3 9.03 mm to (123.0, 175.0)
- moved R56 9.02 mm to (118.8, 190.2), turned to 180 degrees
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
Commit message: breaking for night
Parts:
- moved C1 0.50 mm to (89.2, 189.8)
- moved C3 0.50 mm to (122.8, 181.8)
- moved C4 0.50 mm to (110.8, 181.8)
- moved C6 0.50 mm to (93.0, 189.8)
- moved D33 0.50 mm to (102.0, 186.2)
- moved D35 0.50 mm to (102.0, 183.2)
- moved D36 0.50 mm to (102.0, 189.2)
- moved Q1 0.50 mm to (130.8, 184.8)
- moved Q2 0.50 mm to (97.2, 184.8)
- moved R48 0.50 mm to (114.8, 185.8)
- moved R49 0.50 mm to (126.8, 187.8)
- moved R50 0.50 mm to (126.8, 185.8)
- moved R51 0.50 mm to (106.8, 189.8)
- moved R52 0.50 mm to (126.8, 181.8)
- moved R53 0.50 mm to (126.8, 189.8)
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