File: Wasp_Hive.sch (KiCad schematic (older format))
At the start: 125 parts, among them J0 WASP_OUT, J1 WASP_OUT, J10 WASP_OUT, J11 WASP_OUT, J12 WASP_OUT, J13 WASP_OUT, J14 WASP_OUT, J15 WASP_OUT, J16 FM_IN, J17 DENS_IN, J18 DENS_IN, J2 WASP_OUT, J3 WASP_OUT, J4 WASP_OUT, J5 WASP_OUT, J6 WASP_OUT, J7 WASP_OUT, J8 WASP_OUT, J9 WASP_OUT, Q1 MMBT3904, Q2 MMBT3904, U0 74HC245, U1 74HC245, U2 MCP6002-xP, U3 L78M05ABDT-TR, U4 MCP6002-xP, U5 TEENSY_3.2_MINIMAL

Commit message: first form factor
Parts:
- removed J18: DENS_IN, HammerheadAudio:EuroJack_MonoSW_THT_NOREF_Mask, symbol Connector:EuroJack_Mono_3.5mm_Switched
- D0, D10, D12, D14, D16, D18, D2, D20, D22, D24, D26, D28, D30, D4, D6, D8: footprint HammerheadAudio:Backlit_Larvae_Smaller -> LED_SMD:LED_1206_3216Metric_Pad1.42x1.75mm_HandSolder
- R48, R49, R50, R51, R52, R53, R54: footprint Resistor_SMD:R_0603_1608Metric_Pad1.05x0.95mm_HandSolder_SmallRef -> HammerheadAudio:R_THT_P7.62_Centered
- U0, U1: footprint Package_SO:SO-20_12.8x7.5mm_P1.27mm -> Package_DIP:DIP-20_W7.62mm_Socket
- U2, U4: footprint Package_SO:SOIC-8_3.9x4.9mm_P1.27mm -> Package_DIP:DIP-8_W7.62mm_Socket
Connections:
- net DENSITY_CV: now also R54.1, U4.1

Commit message: alterantive sketch
Parts:
- removed D32, D34: SM4007PL, Diode_SMD:D_SOD-123, symbol Device:D
- removed J16: FM_IN, HammerheadAudio:EuroJack_MonoSW_THT_NOREF_Mask, symbol Connector:EuroJack_Mono_3.5mm_Switched
- removed Q1: MMBT3904, Package_TO_SOT_SMD:SOT-23, symbol Transistor_BJT:MMBT3904
- removed R48, R49: 100k, HammerheadAudio:R_THT_P7.62_Centered, symbol Device:R
- removed R50: 1k, HammerheadAudio:R_THT_P7.62_Centered, symbol Device:R
- removed unit 1 of U2
- renumbered U4 to U2, U5 to U4
Connections:
- net DENSITY_CV: no longer R54.1, U2.1
- net T0: now also U4.0 (0_RX1_Touch)
- net T1: now also U4.1 (1_TX1_Touch)
- net T10: now also U4.10 (10_TX2_CS0_PWM)
- net T11: now also U4.11 (11_MOSI0)
- net T12: now also U4.12 (12_MISO0)
- net T13: now also U4.14 (14_A0_SCK)
- net T14: now also U4.15 (15_A1_CS_Touch)
- net T15: now also U4.16 (16_A2_SCL0_Touch)
- net T2: now also U4.2
- net T3: now also U4.3 (3_TX_PWM)
- net T4: now also U4.4 (4_RX_PWM)
- net T5: now also U4.5 (5_TX1_PWM)
- net T6: now also U4.6 (6_PWM)
- net T7: now also U4.7 (7_RX3_DOUT)
- net T8: now also U4.8 (8_TX3_DIN)
- net T9: now also U4.9 (9_RX2_CS_PWM)
- net DENS_NORM: no longer names the net of J17.3
- net DENS_NORM: now also R54.1, U2.1
- no-connect marks 24 -> 23
Other:
- moved on the sheet: R52, R54, U2A

Commit message: Finished schematic
Parts:
- removed Q2: MMBT3904, Package_TO_SOT_SMD:SOT-23, symbol Transistor_BJT:MMBT3904
- removed RV2: MIN_FREQ, Crossley_Footprints:SMD_TRIM_JLC, symbol Device:R_POT_TRIM
- removed RV5: MAX_FREQ, Crossley_Footprints:SMD_TRIM_JLC, symbol Device:R_POT_TRIM
- added C3, C4: 0.1uf, Capacitor_SMD:C_0603_1608Metric_Pad1.05x0.95mm_HandSolder_SmallRef, symbol Device:C
- added D32: DENS, LED_SMD:LED_1206_3216Metric_Pad1.42x1.75mm_HandSolder, symbol Device:LED
- added D34: DROP, LED_SMD:LED_1206_3216Metric_Pad1.42x1.75mm_HandSolder, symbol Device:LED
- added D36: SM4007PL, Diode_SMD:D_SOD-123, symbol Device:D
- added D37: PANIC, LED_SMD:LED_1206_3216Metric_Pad1.42x1.75mm_HandSolder, symbol Device:LED
- added D38: M7, Diode_SMD:D_SMA, symbol Device:D
- added J16: DENS_OUT, HammerheadAudio:EuroJack_MonoSW_THT_NOREF_Mask, symbol Connector:EuroJack_Mono_3.5mm_Switched
- added J18: DROP_OUT, HammerheadAudio:EuroJack_MonoSW_THT_NOREF_Mask, symbol Connector:EuroJack_Mono_3.5mm_Switched
- added J19: PANIC_IN, HammerheadAudio:EuroJack_MonoSW_THT_NOREF_Mask, symbol Connector:EuroJack_Mono_3.5mm_Switched
- added J20, J21, J22, J23, J24: GND, HammerheadAudio:M3_Plated, symbol Connector:Conn_01x01_Female
- added J25: PWR, HammerheadAudio:M3_Plated, symbol Connector:Conn_01x01_Female
- added Q1: 2N3904, HammerheadAudio:TO-92_Inline_Centered, symbol Transistor_BJT:2N3904
- added R48, R55, R60: 1k, Resistor_SMD:R_0603_1608Metric_Pad1.05x0.95mm_HandSolder_SmallRef, symbol Device:R
- added R49, R50, R56, R61: 100k, Resistor_SMD:R_0603_1608Metric_Pad1.05x0.95mm_HandSolder_SmallRef (at -2.794 0)_ (descr _STANDOFF (#4 SCREW)_)_ (tags _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, symbol Device:R
- added R57: 47k, Resistor_SMD:R_0603_1608Metric_Pad1.05x0.95mm_HandSolder_SmallRef, symbol Device:R
- added R58, R62: GP_R, Resistor_SMD:R_0603_1608Metric_Pad1.05x0.95mm_HandSolder_SmallRef, symbol Device:R
- added R59: WSP_R, Resistor_SMD:R_0603_1608Metric_Pad1.05x0.95mm_HandSolder_SmallRef, symbol Device:R
- added RV4: XCTRL, Crossley_Footprints:SMD_TRIM_JLC, symbol Device:R_POT_TRIM
- added unit 1 of U2
- added unit 3 of U2
- added unit 2 of U3
- added unit 3 of U3
- R51, R52, R53, R54: footprint HammerheadAudio:R_THT_P7.62_Centered -> Resistor_SMD:R_0603_1608Metric_Pad1.05x0.95mm_HandSolder_SmallRef (at -2.794 0)_ (descr _STANDOFF (#4 SCREW)_)_ (tags _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
- renumbered RV4 to RV2, U2 to U3, U3 to U5
Connections:
- net DENSITY_CV is gone; now on net DENS_CV: U2.6 (-), U2.7
- net DENS_OUT is gone; now on net DENS_INTERNAL: U3.3 (+)
- net +3V3: now also U4.3V (3.3V_max100mA), R62.2, RV4.3
- net +5V: now also C4.1, U2.8 (V+)
- net GND: now also U4.GND1 (GND), C3.2, C4.2, D32.1 (K), D34.1 (K), D38.2 (A), J16.2, J18.2, J19.2, J20.1 (Pin_1), J21.1 (Pin_1), J22.1 (Pin_1), J23.1 (Pin_1), J24.1 (Pin_1), Q1.1 (E), R49.1, R56.1, R61.2, RV4.1, U2.4 (V-), U3.4 (V-)
- net MAX_DENS: now also U4.18 (18_A4_SDA0_Touch)
- net MIN_DENS: now also U4.17 (17_A3_SDA0_Touch)
- net ROC: now also U4.19 (19_A5_SCL0_Touch)
- net VDD: now also C3.1, D38.1 (K), J25.1 (Pin_1), U3.8 (V+)
- net DROP: now reaches U4.13 (13_LED_SCK0)
- net DROP: now also U2.3 (+)
- net DENS_CV: now reaches U4.20 (20_A6_CS_PWM)
- net DENS_CV: now also U3.5 (+)
- net PANIC: now reaches U4.21 (21_A7_RX1_CS_PWM)
- net PANIC: now also D37.1 (K), Q1.3 (C)
- net DENS_IND: now reaches U4.22 (22_A8_Touch_PWM)
- net DENS_IND: now also R58.2
- net XCTRL: now reaches U4.23 (23_A9_Touch_PWM)
- net XCTRL: now also RV4.2
- net DENS_INTERNAL: now reaches U4.A12 (A14/DAC)
- net at R54.1, U3.1: now also R48.1; no longer J17.3
- new net: J17.3, R48.2
- new net: D36.1 (K), Q1.2 (B), R61.1
- new net: D36.2 (A), R60.1
- new net: J19.1, R60.2
- new net: D37.2 (A), R62.1
- new net: R50.1, R55.1, U3.7
- new net: R49.2, R50.2, U3.6 (-)
- new net: J16.1, R55.2
- new net: J18.1, R57.1, R59.2, U2.1
- new net: R56.2, R57.2, U2.2 (-)
- new net: D32.2 (A), R58.1
- new net: D34.2 (A), R59.1
- no-connect marks 23 -> 27
Other:
- moved on the sheet: C1, C2, D0, D1, D10, D11, D12, D13, D14, D15, D16, D17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

Commit message: layout ideas
Parts:
- removed Q1: 2N3904, HammerheadAudio:TO-92_Inline_Centered, symbol Transistor_BJT:2N3904
- added C5, C6: 0.1uf, Capacitor_SMD:C_0603_1608Metric_Pad1.05x0.95mm_HandSolder_SmallRef_Fab, symbol Device:C
- added D39: DENS2, LED_SMD:LED_1206_3216Metric_Pad1.42x1.75mm_HandSolder_FabRef, symbol Device:LED
- added D40: DENS3, LED_SMD:LED_1206_3216Metric_Pad1.42x1.75mm_HandSolder_FabRef, symbol Device:LED
- added D41: DROP2, LED_SMD:LED_1206_3216Metric_Pad1.42x1.75mm_HandSolder_FabRef, symbol Device:LED
- added Q1, Q2: MMBT3904, Package_TO_SOT_SMD:SOT-23, symbol Transistor_BJT:MMBT3904
- added R63, R67: 1k, Resistor_SMD:R_0603_1608Metric_Pad1.05x0.95mm_HandSolder_SmallRef_Fab, symbol Device:R
- added R64, R65: DENS_R, Resistor_SMD:R_0603_1608Metric_Pad1.05x0.95mm_HandSolder_SmallRef_Fab, symbol Device:R
- added R66: WSP_R, Resistor_SMD:R_0603_1608Metric_Pad1.05x0.95mm_HandSolder_SmallRef_Fab, symbol Device:R
- added SW1: SW_SPDT, HammerheadAudio:Tayda_Slide_SPDT, symbol Switch:SW_SPDT
- C1, C2, C3, C4: footprint Capacitor_SMD:C_0603_1608Metric_Pad1.05x0.95mm_HandSolder_SmallRef -> Capacitor_SMD:C_0603_1608Metric_Pad1.05x0.95mm_HandSolder_SmallRef_Fab
- D0, D10, D12, D14, D16, D18, D2, D20, D22, D24, D26, D28, D30, D4, D6, D8: footprint LED_SMD:LED_1206_3216Metric_Pad1.42x1.75mm_HandSolder -> HammerheadAudio:Backlit_Larvae_Smaller
- D1, D11, D13, D15, D17, D19, D21, D23, D25, D27, D29, D3, D31, D34, D37, D5, D7, D9: footprint LED_SMD:LED_1206_3216Metric_Pad1.42x1.75mm_HandSolder -> LED_SMD:LED_1206_3216Metric_Pad1.42x1.75mm_HandSolder_FabRef
- D32: value DENS -> DENS1; footprint LED_SMD:LED_1206_3216Metric_Pad1.42x1.75mm_HandSolder -> LED_SMD:LED_1206_3216Metric_Pad1.42x1.75mm_HandSolder_FabRef
- R0, R1, R10, R11, R12, R13, R14, R15, R16, R17, R18, R19, R2, R20, R21, R22, R23, R24, R25, R26, R27, R28, R29, R3, R30, R31, R32, R33, R34, R35, R36, R37, R38, R39, R4, R40, R41, R42, R43, R44, R45, R46, R47, R48, R5, R55, R57, R59, R6, R60, R62, R7, R8, R9: footprint Resistor_SMD:R_0603_1608Metric_Pad1.05x0.95mm_HandSolder_SmallRef -> Resistor_SMD:R_0603_1608Metric_Pad1.05x0.95mm_HandSolder_SmallRef_Fab
- R49, R50, R51, R52, R53, R54, R56, R61: footprint Resistor_SMD:R_0603_1608Metric_Pad1.05x0.95mm_HandSolder_SmallRef (at -2.794 0)_ (descr _STANDOFF (#4 SCREW)_)_ (tags _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 -> Resistor_SMD:R_0603_1608Metric_Pad1.05x0.95mm_HandSolder_SmallRef_Fab
- R58: value GP_R -> DENS_R; footprint Resistor_SMD:R_0603_1608Metric_Pad1.05x0.95mm_HandSolder_SmallRef -> Resistor_SMD:R_0603_1608Metric_Pad1.05x0.95mm_HandSolder_SmallRef_Fab
- U0, U1: footprint Package_DIP:DIP-20_W7.62mm_Socket -> Package_SO:SOIC-20W_7.5x12.8mm_P1.27mm
- U2, U3: footprint Package_DIP:DIP-8_W7.62mm_Socket -> Package_SO:SOIC-8_3.9x4.9mm_P1.27mm
- U4: footprint MeowWolf_Templates:TEENSY_LC_NO_SILK -> MeowWolf_Templates:TEENSY_LC_MIN_SILK_2SIDE
Connections:
- net +3V3: now also C4.1, U2.8 (V+)
- net +5V: now also C5.1, C6.1; no longer C4.1, U0.1 (A->B), U1.1 (A->B), U2.8 (V+)
- net DENS_IND: now also R63.1; no longer R58.2
- net GND: now also U0.1 (A->B), U1.1 (A->B), C5.2, C6.2, D41.1 (K), Q1.2 (E), Q2.2 (E); no longer D32.1 (K)
- net O0: now also U0.2 (A0); no longer U0.18 (B0)
- net O1: now also U0.3 (A1); no longer U0.17 (B1)
- net O10: now also U1.4 (A2); no longer U1.16 (B2)
- net O11: now also U1.5 (A3); no longer U1.15 (B3)
- net O12: now also U1.6 (A4); no longer U1.14 (B4)
- net O13: now also U1.7 (A5); no longer U1.13 (B5)
- net O14: now also U1.8 (A6); no longer U1.12 (B6)
- net O15: now also U1.9 (A7); no longer U1.11 (B7)
- net O2: now also U0.4 (A2); no longer U0.16 (B2)
- net O3: now also U0.5 (A3); no longer U0.15 (B3)
- net O4: now also U0.6 (A4); no longer U0.14 (B4)
- net O5: now also U0.7 (A5); no longer U0.13 (B5)
- net O6: now also U0.8 (A6); no longer U0.12 (B6)
- net O7: now also U0.9 (A7); no longer U0.11 (B7)
- net O8: now also U1.2 (A0); no longer U1.18 (B0)
- net O9: now also U1.3 (A1); no longer U1.17 (B1)
- net PANIC: now also Q2.3 (C)
- net T0: now also U0.18 (B0), U4.14 (14_A0_SCK); no longer U0.2 (A0), U4.0 (0_RX1_Touch)
- net T1: now also U0.17 (B1), U4.15 (15_A1_CS_Touch); no longer U0.3 (A1), U4.1 (1_TX1_Touch)
- net T10: now also U1.16 (B2), U4.5 (5_TX1_PWM); no longer U1.4 (A2), U4.10 (10_TX2_CS0_PWM)
- net T11: now also U1.15 (B3), U4.4 (4_RX_PWM); no longer U1.5 (A3), U4.11 (11_MOSI0)
- net T12: now also U1.14 (B4), U4.3 (3_TX_PWM); no longer U1.6 (A4), U4.12 (12_MISO0)
- net T13: now also U1.13 (B5), U4.2; no longer U1.7 (A5), U4.14 (14_A0_SCK)
- net T14: now also U1.12 (B6), U4.1 (1_TX1_Touch); no longer U1.8 (A6), U4.15 (15_A1_CS_Touch)
- net T15: now also U1.11 (B7), U4.0 (0_RX1_Touch); no longer U1.9 (A7), U4.16 (16_A2_SCL0_Touch)
- net T2: now also U0.16 (B2), U4.16 (16_A2_SCL0_Touch); no longer U0.4 (A2), U4.2
- net T3: now also U0.15 (B3), U4.12 (12_MISO0); no longer U0.5 (A3), U4.3 (3_TX_PWM)
- net T4: now also U0.14 (B4), U4.11 (11_MOSI0); no longer U0.6 (A4), U4.4 (4_RX_PWM)
- net T5: now also U0.13 (B5), U4.10 (10_TX2_CS0_PWM); no longer U0.7 (A5), U4.5 (5_TX1_PWM)
- net T6: now also U0.12 (B6), U4.9 (9_RX2_CS_PWM); no longer U0.8 (A6), U4.6 (6_PWM)
- net T7: now also U0.11 (B7), U4.8 (8_TX3_DIN); no longer U0.9 (A7), U4.7 (7_RX3_DOUT)
- net T8: now also U1.18 (B0), U4.7 (7_RX3_DOUT); no longer U1.2 (A0), U4.8 (8_TX3_DIN)
- net T9: now also U1.17 (B1), U4.6 (6_PWM); no longer U1.3 (A1), U4.9 (9_RX2_CS_PWM)
- net VDD: now also R58.2, R64.2, R65.2, SW1.1 (A); no longer J25.1 (Pin_1)
- net at D36.1 (K), R61.1: now also Q2.1 (B)
- net at R57.1, R59.2, U2.1: now also R66.2, R67.1; no longer J18.1
- new net: D41.2 (A), R66.1
- new net: Q1.1 (B), R63.2
- new net: D39.2 (A), R64.1
- new net: D32.1 (K), D39.1 (K), D40.1 (K), Q1.3 (C)
- new net: D40.2 (A), R65.1
- new net: J25.1 (Pin_1), SW1.2 (B)
- new net: J18.1, R67.2
- no-connect marks 27 -> 28
Other:
- moved on the sheet: D32, D38, J20, J21, J22, J23, J24, J25, R58

Commit message: layout progress
Connections:
- net +3V3: no longer C4.1, U2.8 (V+)
- net +5V: now also C4.1, U2.8 (V+)
- net DENS_CV: now also U2.1, U2.2 (-); no longer U2.6 (-), U2.7
- net DROP: now also U2.5 (+); no longer U2.3 (+)
- net at R57.1, R59.2, R66.2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: now also U2.7; no longer U2.1
- net at D33.1 (K), D35.2 (A), R51.1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: now also U2.3 (+); no longer U2.5 (+)
- net at R56.2, R57.2: now also U2.6 (-); no longer U2.2 (-)
Other:
- moved on the sheet: RV1, RV2, RV3, RV4, U2A, U2B
Changed lines of the file:
@@
 L power:+3.3V #PWR0112
 U 1 1 629E6C8F
-P 13100 4150
-F 0 "#PWR0112" H 13100 4000 50  0001 C CNN
-F 1 "+3.3V" H 13115 4323 50  0000 C CNN
-F 2 "" H 13100 4150 50  0001 C CNN
-F 3 "" H 13100 4150 50  0001 C CNN
-	1    13100 4150
+P 12100 4100
+F 0 "#PWR0112" H 12100 3950 50  0001 C CNN
+F 1 "+3.3V" H 12115 4273 50  0000 C CNN
+F 2 "" H 12100 4100 50  0001 C CNN
+F 3 "" H 12100 4100 50  0001 C CNN
+	1    12100 4100
 	0    1    1    0
 $EndComp
@@
 L power:GND #PWR0113
 U 1 1 629E7E3D
-P 12700 4150
-F 0 "#PWR0113" H 12700 3900 50  0001 C CNN
-F 1 "GND" H 12705 3977 50  0000 C CNN
-F 2 "" H 12700 4150 50  0001 C CNN
-F 3 "" H 12700 4150 50  0001 C CNN
-	1    12700 4150
-	0    1    1    0
-$EndComp
-Wire Wire Line
-	12700 4150 12750 4150
-Wire Wire Line
-	13050 4150 13100 4150
+P 11700 4100
+F 0 "#PWR0113" H 11700 3850 50  0001 C CNN
+F 1 "GND" H 11705 3927 50  0000 C CNN
+F 2 "" H 11700 4100 50  0001 C CNN
+F 3 "" H 11700 4100 50  0001 C CNN
+	1    11700 4100
+	0    1    1    0
+$EndComp
+Wire Wire Line
+	11700 4100 11750 4100
+Wire Wire Line
+	12050 4100 12100 4100
 $Comp
 L power:+3.3V #PWR0114
 U 1 1 62A67403
-P 14050 4150
-F 0 "#PWR0114" H 14050 4000 50  0001 C CNN
-F 1 "+3.3V" H 14065 4323 50  0000 C CNN
-F 2 "" H 14050 4150 50  0001 C CNN
-F 3 "" H 14050 4150 50  0001 C CNN
-	1    14050 4150
+P 13050 4100
+F 0 "#PWR0114" H 13050 3950 50  0001 C CNN
+F 1 "+3.3V" H 13065 4273 50  0000 C CNN
+F 2 "" H 13050 4100 50  0001 C CNN
+F 3 "" H 13050 4100 50  0001 C CNN
+	1    13050 4100
 	0    1    1    0
 $EndComp
@@
 L power:GND #PWR0115
 U 1 1 62A6740D
-P 13650 4150
-F 0 "#PWR0115" H 13650 3900 50  0001 C CNN
-F 1 "GND" H 13655 3977 50  0000 C CNN
-F 2 "" H 13650 4150 50  0001 C CNN
-F 3 "" H 13650 4150 50  0001 C CNN
-	1    13650 4150
-	0    1    1    0
-$EndComp
-Wire Wire Line
-	13650 4150 13700 4150
-Wire Wire Line
-	14000 4150 14050 4150
+P 12650 4100
+F 0 "#PWR0115" H 12650 3850 50  0001 C CNN
+F 1 "GND" H 12655 3927 50  0000 C CNN
+F 2 "" H 12650 4100 50  0001 C CNN
+F 3 "" H 12650 4100 50  0001 C CNN
+	1    12650 4100
+	0    1    1    0
+$EndComp
+Wire Wire Line
+	12650 4100 12700 4100
+Wire Wire Line
+	13000 4100 13050 4100
 $Comp
 L power:+3.3V #PWR0120
 U 1 1 62B0F4B3
-P 14950 4150
-F 0 "#PWR0120" H 14950 4000 50  0001 C CNN
-F 1 "+3.3V" H 14965 4323 50  0000 C CNN
-F 2 "" H 14950 4150 50  0001 C CNN
-F 3 "" H 14950 4150 50  0001 C CNN
-	1    14950 4150
+P 13950 4100
+F 0 "#PWR0120" H 13950 3950 50  0001 C CNN
+F 1 "+3.3V" H 13965 4273 50  0000 C CNN
+F 2 "" H 13950 4100 50  0001 C CNN
+F 3 "" H 13950 4100 50  0001 C CNN
+	1    13950 4100
 	0    1    1    0
 $EndComp
@@
 L power:GND #PWR0121
 U 1 1 62B0F4BD
-P 14550 4150
-F 0 "#PWR0121" H 14550 3900 50  0001 C CNN
-F 1 "GND" H 14555 3977 50  0000 C CNN
-F 2 "" H 14550 4150 50  0001 C CNN
-F 3 "" H 14550 4150 50  0001 C CNN
-	1    14550 4150
-	0    1    1    0
-$EndComp
-Wire Wire Line
-	14550 4150 14600 4150
-Wire Wire Line
-	14900 4150 14950 4150
-Text GLabel 12900 4350 3    50   Input ~ 0
+P 13550 4100
+F 0 "#PWR0121" H 13550 3850 50  0001 C CNN
+F 1 "GND" H 13555 3927 50  0000 C CNN
+F 2 "" H 13550 4100 50  0001 C CNN
+F 3 "" H 13550 4100 50  0001 C CNN
+	1    13550 4100
+	0    1    1    0
+$EndComp
+Wire Wire Line
+	13550 4100 13600 4100
+Wire Wire Line
+	13900 4100 13950 4100
+Text GLabel 11900 4300 3    50   Input ~ 0
 MIN_DENS
-Text GLabel 13850 4350 3    50   Input ~ 0
+Text GLabel 12850 4300 3    50   Input ~ 0
 MAX_DENS
 Wire Wire Line
-	12900 4300 12900 4350
-Wire Wire Line
-	13850 4300 13850 4350
-Text GLabel 14750 4350 3    50   Input ~ 0
+	11900 4250 11900 4300
+Wire Wire Line
+	12850 4250 12850 4300
+Text GLabel 13750 4300 3    50   Input ~ 0
 ROC
 Wire Wire Line
-	14750 4300 14750 4350
+	13750 4250 13750 4300
 Wire Wire Line
 	7350 7850 7350 7900
@@
 L Device:R_POT_TRIM RV3
 U 1 1 62B0F4A9
-P 14750 4150
-F 0 "RV3" V 14543 4150 50  0000 C CNN
-F 1 "CHANGE_RATE" V 14634 4150 50  0000 C CNN
-F 2 "Crossley_Footprints:SMD_TRIM_JLC" H 14750 4150 50  0001 C CNN
-F 3 "~" H 14750 4150 50  0001 C CNN
-	1    14750 4150
+P 13750 4100
+F 0 "RV3" V 13543 4100 50  0000 C CNN
+F 1 "CHANGE_RATE" V 13634 4100 50  0000 C CNN
+F 2 "Crossley_Footprints:SMD_TRIM_JLC" H 13750 4100 50  0001 C CNN
+F 3 "~" H 13750 4100 50  0001 C CNN
+	1    13750 4100
 	0    -1   1    0
 $EndComp
@@
 L Device:R_POT_TRIM RV2
 U 1 1 62A673F9
-P 13850 4150
-F 0 "RV2" V 13643 4150 50  0000 C CNN
-F 1 "MAX_DENS" V 13734 4150 50  0000 C CNN
-F 2 "Crossley_Footprints:SMD_TRIM_JLC" H 13850 4150 50  0001 C CNN
-F 3 "~" H 13850 4150 50  0001 C CNN
-	1    13850 4150
+P 12850 4100
+F 0 "RV2" V 12643 4100 50  0000 C CNN
+F 1 "MAX_DENS" V 12734 4100 50  0000 C CNN
+F 2 "Crossley_Footprints:SMD_TRIM_JLC" H 12850 4100 50  0001 C CNN
+F 3 "~" H 12850 4100 50  0001 C CNN
+	1    12850 4100
 	0    -1   1    0
 $EndComp
@@
 L Device:R_POT_TRIM RV1
 U 1 1 629E5FAE
-P 12900 4150
-F 0 "RV1" V 12693 4150 50  0000 C CNN
-F 1 "MIN_DENS" V 12784 4150 50  0000 C CNN
-F 2 "Crossley_Footprints:SMD_TRIM_JLC" H 12900 4150 50  0001 C CNN
-F 3 "~" H 12900 4150 50  0001 C CNN
-	1    12900 4150
+P 11900 4100
+F 0 "RV1" V 11693 4100 50  0000 C CNN
+F 1 "MIN_DENS" V 11784 4100 50  0000 C CNN
+F 2 "Crossley_Footprints:SMD_TRIM_JLC" H 11900 4100 50  0001 C CNN
+F 3 "~" H 11900 4100 50  0001 C CNN
+	1    11900 4100
 	0    -1   1    0
 $EndComp
@@
 L Amplifier_Operational:MCP6002-xP U2
 U 2 1 62548586
-P 9250 5700
-F 0 "U2" H 9250 5333 50  0000 C CNN
-F 1 "MCP6002-xP" H 9250 5424 50  0000 C CNN
-F 2 "Package_SO:SOIC-8_3.9x4.9mm_P1.27mm" H 9250 5700 50  0001 C CNN
-F 3 "C7377" H 9250 5700 50  0001 C CNN
-	2    9250 5700
-	1    0    0    1
+P 12800 5750
+F 0 "U2" H 12800 5383 50  0000 C CNN
+F 1 "MCP6002-xP" H 12800 5474 50  0000 C CNN
+F 2 "Package_SO:SOIC-8_3.9x4.9mm_P1.27mm" H 12800 5750 50  0001 C CNN
+F 3 "C7377" H 12800 5750 50  0001 C CNN
+	2    12800 5750
+	1    0    0    -1
 $EndComp
 $Comp
@@
 L Amplifier_Operational:MCP6002-xP U2
 U 1 1 641C0166
-P 12800 5750
-F 0 "U2" H 12800 5383 50  0000 C CNN
-F 1 "MCP6002-xP" H 12800 5474 50  0000 C CNN
-F 2 "Package_SO:SOIC-8_3.9x4.9mm_P1.27mm" H 12800 5750 50  0001 C CNN
-F 3 "C7377" H 12800 5750 50  0001 C CNN
-	1    12800 5750
-	1    0    0    -1
+P 9250 5700
+F 0 "U2" H 9250 5333 50  0000 C CNN
+F 1 "MCP6002-xP" H 9250 5424 50  0000 C CNN
+F 2 "Package_SO:SOIC-8_3.9x4.9mm_P1.27mm" H 9250 5700 50  0001 C CNN
+F 3 "C7377" H 9250 5700 50  0001 C CNN
+	1    9250 5700
+	1    0    0    1
 $EndComp
 Wire Wire Line
@@
 L power:+3.3V #PWR023
 U 1 1 648E25AC
-P 12150 4150
-F 0 "#PWR023" H 12150 4000 50  0001 C CNN
-F 1 "+3.3V" H 12165 4323 50  0000 C CNN
-F 2 "" H 12150 4150 50  0001 C CNN
-F 3 "" H 12150 4150 50  0001 C CNN
-	1    12150 4150
+P 14800 4100
+F 0 "#PWR023" H 14800 3950 50  0001 C CNN
+F 1 "+3.3V" H 14815 4273 50  0000 C CNN
+F 2 "" H 14800 4100 50  0001 C CNN
+F 3 "" H 14800 4100 50  0001 C CNN
+	1    14800 4100
 	0    1    1    0
 $EndComp
@@
 L power:GND #PWR022
 U 1 1 648E25B6
-P 11750 4150
-F 0 "#PWR022" H 11750 3900 50  0001 C CNN
-F 1 "GND" H 11755 3977 50  0000 C CNN
-F 2 "" H 11750 4150 50  0001 C CNN
-F 3 "" H 11750 4150 50  0001 C CNN
-	1    11750 4150
-	0    1    1    0
-$EndComp
-Wire Wire Line
-	11750 4150 11800 4150
-Wire Wire Line
-	12100 4150 12150 4150
-Text GLabel 11950 4350 3    50   Input ~ 0
+P 14400 4100
+F 0 "#PWR022" H 14400 3850 50  0001 C CNN
+F 1 "GND" H 14405 3927 50  0000 C CNN
+F 2 "" H 14400 4100 50  0001 C CNN
+F 3 "" H 14400 4100 50  0001 C CNN
+	1    14400 4100
+	0    1    1    0
+$EndComp
+Wire Wire Line
+	14400 4100 14450 4100
+Wire Wire Line
+	14750 4100 14800 4100
+Text GLabel 14600 4300 3    50   Input ~ 0
 XCTRL
 Wire Wire Line
-	11950 4300 11950 4350
+	14600 4250 14600 4300
 $Comp
 L Device:R_POT_TRIM RV4
 U 1 1 648E25C4
-P 11950 4150
-F 0 "RV4" V 11743 4150 50  0000 C CNN
-F 1 "XCTRL" V 11834 4150 50  0000 C CNN
-F 2 "Crossley_Footprints:SMD_TRIM_JLC" H 11950 4150 50  0001 C CNN
-F 3 "~" H 11950 4150 50  0001 C CNN
-	1    11950 4150
+P 14600 4100
+F 0 "RV4" V 14393 4100 50  0000 C CNN
+F 1 "XCTRL" V 14484 4100 50  0000 C CNN
+F 2 "Crossley_Footprints:SMD_TRIM_JLC" H 14600 4100 50  0001 C CNN
+F 3 "~" H 14600 4100 50  0001 C CNN
+	1    14600 4100
 	0    -1   1    0
 $EndComp
@@
 	13600 6350 13850 6350
 $Comp
-L power:+3.3V #PWR0124
-U 1 1 624B995D
-P 9650 9900
-F 0 "#PWR0124" H 9650 9750 50  0001 C CNN
-F 1 "+3.3V" H 9665 10073 50  0000 C CNN
-F 2 "" H 9650 9900 50  0001 C CNN
-F 3 "" H 9650 9900 50  0001 C CNN
-	1    9650 9900
-	1    0    0    -1
-$EndComp
-$Comp
 L Device:C C5
 U 1 1 624DF78A
@@
 Wire Wire Line
 	14450 1950 14950 1950
+$Comp
+L power:+5V #PWR0124
+U 1 1 61A7D3BA
+P 9650 9900
+F 0 "#PWR0124" H 9650 9750 50  0001 C CNN
+F 1 "+5V" V 9665 10028 50  0000 L CNN
+F 2 "" H 9650 9900 50  0001 C CNN
+F 3 "" H 9650 9900 50  0001 C CNN
+	1    9650 9900
+	1    0    0    -1
+$EndComp
 $EndSCHEMATC
