File: Wasp_Hive.sch (KiCad schematic (older format))
At the start: 155 parts, among them J0 WASP_OUT, J1 WASP_OUT, J10 WASP_OUT, J11 WASP_OUT, J12 WASP_OUT, J13 WASP_OUT, J14 WASP_OUT, J15 WASP_OUT, J16 DENS_OUT, J17 DENS_IN, J18 DROP_OUT, J19 PANIC_IN, J2 WASP_OUT, J20 GND, J21 GND, J22 GND, J23 GND, J24 GND, J25 PWR, J3 WASP_OUT, J4 WASP_OUT, J5 WASP_OUT, J6 WASP_OUT, J7 WASP_OUT, J8 WASP_OUT, J9 WASP_OUT, Q1 MMBT3904, Q2 MMBT3904, SW1 SW_SPDT, U0 74HC245, U1 74HC245, U2 MCP6002-xP, U3 MCP6002-xP, U4 TEENSY_3.2_MINIMAL, U5 L78M05ABDT-TR

Commit message: footprint update
Parts:
- added J26, J27: GND, HammerheadAudio:M3_Plated, symbol Connector:Conn_01x01_Female
- J0, J1, J10, J11, J12, J13, J14, J15, J2, J3, J4, J5, J6, J7, J8, J9: footprint HammerheadAudio:EuroJack_Hex -> HammerheadAudio:EuroJack_Hex_SmallHoles_NoSilk
- J16, J17, J18, J19: footprint HammerheadAudio:EuroJack_MonoSW_THT_NOREF_Mask -> HammerheadAudio:EuroJack_MonoSW_THT_NOREF_Mask_SmallHoles_NoSilk
Connections:
- net GND: now also J26.1 (Pin_1), J27.1 (Pin_1)
Changed lines of the file:
@@
 F 0 "J17" H 7878 6025 50  0000 C CNN
 F 1 "DENS_IN" H 7878 5934 50  0000 C CNN
-F 2 "HammerheadAudio:EuroJack_MonoSW_THT_NOREF_Mask" H 7850 5800 50  0001 C CNN
+F 2 "HammerheadAudio:EuroJack_MonoSW_THT_NOREF_Mask_SmallHoles_NoSilk" H 7850 5800 50  0001 C CNN
 F 3 "~" H 7850 5800 50  0001 C CNN
 	1    7850 5800
@@
 F 0 "J15" H 5628 8825 50  0000 C CNN
 F 1 "WASP_OUT" H 5628 8734 50  0000 C CNN
-F 2 "HammerheadAudio:EuroJack_Hex" H 5600 8600 50  0001 C CNN
+F 2 "HammerheadAudio:EuroJack_Hex_SmallHoles_NoSilk" H 5600 8600 50  0001 C CNN
 F 3 "~" H 5600 8600 50  0001 C CNN
 	1    5600 8600
@@
 F 0 "J14" H 5628 7325 50  0000 C CNN
 F 1 "WASP_OUT" H 5628 7234 50  0000 C CNN
-F 2 "HammerheadAudio:EuroJack_Hex" H 5600 7100 50  0001 C CNN
+F 2 "HammerheadAudio:EuroJack_Hex_SmallHoles_NoSilk" H 5600 7100 50  0001 C CNN
 F 3 "~" H 5600 7100 50  0001 C CNN
 	1    5600 7100
@@
 F 0 "J13" H 5628 5825 50  0000 C CNN
 F 1 "WASP_OUT" H 5628 5734 50  0000 C CNN
-F 2 "HammerheadAudio:EuroJack_Hex" H 5600 5600 50  0001 C CNN
+F 2 "HammerheadAudio:EuroJack_Hex_SmallHoles_NoSilk" H 5600 5600 50  0001 C CNN
 F 3 "~" H 5600 5600 50  0001 C CNN
 	1    5600 5600
@@
 F 0 "J12" H 5628 4325 50  0000 C CNN
 F 1 "WASP_OUT" H 5628 4234 50  0000 C CNN
-F 2 "HammerheadAudio:EuroJack_Hex" H 5600 4100 50  0001 C CNN
+F 2 "HammerheadAudio:EuroJack_Hex_SmallHoles_NoSilk" H 5600 4100 50  0001 C CNN
 F 3 "~" H 5600 4100 50  0001 C CNN
 	1    5600 4100
@@
 F 0 "J11" H 4328 8775 50  0000 C CNN
 F 1 "WASP_OUT" H 4328 8684 50  0000 C CNN
-F 2 "HammerheadAudio:EuroJack_Hex" H 4300 8550 50  0001 C CNN
+F 2 "HammerheadAudio:EuroJack_Hex_SmallHoles_NoSilk" H 4300 8550 50  0001 C CNN
 F 3 "~" H 4300 8550 50  0001 C CNN
 	1    4300 8550
@@
 F 0 "J10" H 4328 7275 50  0000 C CNN
 F 1 "WASP_OUT" H 4328 7184 50  0000 C CNN
-F 2 "HammerheadAudio:EuroJack_Hex" H 4300 7050 50  0001 C CNN
+F 2 "HammerheadAudio:EuroJack_Hex_SmallHoles_NoSilk" H 4300 7050 50  0001 C CNN
 F 3 "~" H 4300 7050 50  0001 C CNN
 	1    4300 7050
@@
 F 0 "J9" H 4328 5775 50  0000 C CNN
 F 1 "WASP_OUT" H 4328 5684 50  0000 C CNN
-F 2 "HammerheadAudio:EuroJack_Hex" H 4300 5550 50  0001 C CNN
+F 2 "HammerheadAudio:EuroJack_Hex_SmallHoles_NoSilk" H 4300 5550 50  0001 C CNN
 F 3 "~" H 4300 5550 50  0001 C CNN
 	1    4300 5550
@@
 F 0 "J8" H 4328 4275 50  0000 C CNN
 F 1 "WASP_OUT" H 4328 4184 50  0000 C CNN
-F 2 "HammerheadAudio:EuroJack_Hex" H 4300 4050 50  0001 C CNN
+F 2 "HammerheadAudio:EuroJack_Hex_SmallHoles_NoSilk" H 4300 4050 50  0001 C CNN
 F 3 "~" H 4300 4050 50  0001 C CNN
 	1    4300 4050
@@
 F 0 "J7" H 2778 8775 50  0000 C CNN
 F 1 "WASP_OUT" H 2778 8684 50  0000 C CNN
-F 2 "HammerheadAudio:EuroJack_Hex" H 2750 8550 50  0001 C CNN
+F 2 "HammerheadAudio:EuroJack_Hex_SmallHoles_NoSilk" H 2750 8550 50  0001 C CNN
 F 3 "~" H 2750 8550 50  0001 C CNN
 	1    2750 8550
@@
 F 0 "J6" H 2778 7275 50  0000 C CNN
 F 1 "WASP_OUT" H 2778 7184 50  0000 C CNN
-F 2 "HammerheadAudio:EuroJack_Hex" H 2750 7050 50  0001 C CNN
+F 2 "HammerheadAudio:EuroJack_Hex_SmallHoles_NoSilk" H 2750 7050 50  0001 C CNN
 F 3 "~" H 2750 7050 50  0001 C CNN
 	1    2750 7050
@@
 F 0 "J5" H 2778 5775 50  0000 C CNN
 F 1 "WASP_OUT" H 2778 5684 50  0000 C CNN
-F 2 "HammerheadAudio:EuroJack_Hex" H 2750 5550 50  0001 C CNN
+F 2 "HammerheadAudio:EuroJack_Hex_SmallHoles_NoSilk" H 2750 5550 50  0001 C CNN
 F 3 "~" H 2750 5550 50  0001 C CNN
 	1    2750 5550
@@
 F 0 "J4" H 2778 4275 50  0000 C CNN
 F 1 "WASP_OUT" H 2778 4184 50  0000 C CNN
-F 2 "HammerheadAudio:EuroJack_Hex" H 2750 4050 50  0001 C CNN
+F 2 "HammerheadAudio:EuroJack_Hex_SmallHoles_NoSilk" H 2750 4050 50  0001 C CNN
 F 3 "~" H 2750 4050 50  0001 C CNN
 	1    2750 4050
@@
 F 0 "J3" H 1478 8725 50  0000 C CNN
 F 1 "WASP_OUT" H 1478 8634 50  0000 C CNN
-F 2 "HammerheadAudio:EuroJack_Hex" H 1450 8500 50  0001 C CNN
+F 2 "HammerheadAudio:EuroJack_Hex_SmallHoles_NoSilk" H 1450 8500 50  0001 C CNN
 F 3 "~" H 1450 8500 50  0001 C CNN
 	1    1450 8500
@@
 F 0 "J2" H 1478 7225 50  0000 C CNN
 F 1 "WASP_OUT" H 1478 7134 50  0000 C CNN
-F 2 "HammerheadAudio:EuroJack_Hex" H 1450 7000 50  0001 C CNN
+F 2 "HammerheadAudio:EuroJack_Hex_SmallHoles_NoSilk" H 1450 7000 50  0001 C CNN
 F 3 "~" H 1450 7000 50  0001 C CNN
 	1    1450 7000
@@
 F 0 "J1" H 1478 5725 50  0000 C CNN
 F 1 "WASP_OUT" H 1478 5634 50  0000 C CNN
-F 2 "HammerheadAudio:EuroJack_Hex" H 1450 5500 50  0001 C CNN
+F 2 "HammerheadAudio:EuroJack_Hex_SmallHoles_NoSilk" H 1450 5500 50  0001 C CNN
 F 3 "~" H 1450 5500 50  0001 C CNN
 	1    1450 5500
@@
 F 0 "J0" H 1478 4225 50  0000 C CNN
 F 1 "WASP_OUT" H 1478 4134 50  0000 C CNN
-F 2 "HammerheadAudio:EuroJack_Hex" H 1450 4000 50  0001 C CNN
+F 2 "HammerheadAudio:EuroJack_Hex_SmallHoles_NoSilk" H 1450 4000 50  0001 C CNN
 F 3 "~" H 1450 4000 50  0001 C CNN
 	1    1450 4000
@@
 F 0 "J16" H 10978 6825 50  0000 C CNN
 F 1 "DENS_OUT" H 10978 6734 50  0000 C CNN
-F 2 "HammerheadAudio:EuroJack_MonoSW_THT_NOREF_Mask" H 10950 6600 50  0001 C CNN
+F 2 "HammerheadAudio:EuroJack_MonoSW_THT_NOREF_Mask_SmallHoles_NoSilk" H 10950 6600 50  0001 C CNN
 F 3 "~" H 10950 6600 50  0001 C CNN
 	1    10950 6600
@@
 F 0 "J18" H 14078 6575 50  0000 C CNN
 F 1 "DROP_OUT" H 14078 6484 50  0000 C CNN
-F 2 "HammerheadAudio:EuroJack_MonoSW_THT_NOREF_Mask" H 14050 6350 50  0001 C CNN
+F 2 "HammerheadAudio:EuroJack_MonoSW_THT_NOREF_Mask_SmallHoles_NoSilk" H 14050 6350 50  0001 C CNN
 F 3 "~" H 14050 6350 50  0001 C CNN
 	1    14050 6350
@@
 F 0 "J19" H 14028 9025 50  0000 C CNN
 F 1 "PANIC_IN" H 14028 8934 50  0000 C CNN
-F 2 "HammerheadAudio:EuroJack_MonoSW_THT_NOREF_Mask" H 14000 8800 50  0001 C CNN
+F 2 "HammerheadAudio:EuroJack_MonoSW_THT_NOREF_Mask_SmallHoles_NoSilk" H 14000 8800 50  0001 C CNN
 F 3 "~" H 14000 8800 50  0001 C CNN
 	1    14000 8800
@@
 L power:GND #PWR026
 U 1 1 64B9B959
-P 7100 4150
-F 0 "#PWR026" H 7100 3900 50  0001 C CNN
-F 1 "GND" H 7105 3977 50  0000 C CNN
-F 2 "" H 7100 4150 50  0001 C CNN
-F 3 "" H 7100 4150 50  0001 C CNN
-	1    7100 4150
+P 7100 5300
+F 0 "#PWR026" H 7100 5050 50  0001 C CNN
+F 1 "GND" H 7105 5127 50  0000 C CNN
+F 2 "" H 7100 5300 50  0001 C CNN
+F 3 "" H 7100 5300 50  0001 C CNN
+	1    7100 5300
 	1    0    0    -1
 $EndComp
@@
 	6950 4050 7100 4050
 Connection ~ 7100 4050
-Wire Wire Line
-	7100 4050 7100 4150
 Wire Wire Line
 	6950 3550 7100 3550
@@
 	1    0    0    -1
 $EndComp
+$Comp
+L Connector:Conn_01x01_Female J26
+U 1 1 61D0182E
+P 6750 4550
+F 0 "J26" H 6642 4325 50  0000 C CNN
+F 1 "GND" H 6642 4416 50  0000 C CNN
+F 2 "HammerheadAudio:M3_Plated" H 6750 4550 50  0001 C CNN
+F 3 "~" H 6750 4550 50  0001 C CNN
+	1    6750 4550
+	-1   0    0    1
+$EndComp
+$Comp
+L Connector:Conn_01x01_Female J27
+U 1 1 61D01838
+P 6750 5050
+F 0 "J27" H 6642 4825 50  0000 C CNN
+F 1 "GND" H 6642 4916 50  0000 C CNN
+F 2 "HammerheadAudio:M3_Plated" H 6750 5050 50  0001 C CNN
+F 3 "~" H 6750 5050 50  0001 C CNN
+	1    6750 5050
+	-1   0    0    1
+$EndComp
+Wire Wire Line
+	7100 4050 7100 4550
+Wire Wire Line
+	6950 5050 7100 5050
+Connection ~ 7100 5050
+Wire Wire Line
+	7100 5050 7100 5300
+Wire Wire Line
+	6950 4550 7100 4550
+Connection ~ 7100 4550
+Wire Wire Line
+	7100 4550 7100 5050
 $EndSCHEMATC

Commit message: layout progress
Parts:
- RV1: value MIN_DENS -> ROC
- RV2: value MAX_DENS -> XCTRL
- RV3: value CHANGE_RATE -> MIN_DENS
- RV4: value XCTRL -> MAX_DENS
Connections:
- net DENS_CV: now also U4.21 (21_A7_RX1_CS_PWM); no longer U4.20 (20_A6_CS_PWM)
- net DENS_IND: now also U4.23 (23_A9_Touch_PWM); no longer U4.22 (22_A8_Touch_PWM)
- net DROP: now also U4.20 (20_A6_CS_PWM); no longer U4.13 (13_LED_SCK0)
- net MAX_DENS: now also RV4.2, U4.19 (19_A5_SCL0_Touch); no longer RV2.2, U4.18 (18_A4_SDA0_Touch)
- net MIN_DENS: now also RV3.2, U4.18 (18_A4_SDA0_Touch); no longer RV1.2, U4.17 (17_A3_SDA0_Touch)
- net PANIC: now also U4.22 (22_A8_Touch_PWM); no longer U4.21 (21_A7_RX1_CS_PWM)
- net ROC: now also RV1.2, U4.16 (16_A2_SCL0_Touch); no longer RV3.2, U4.19 (19_A5_SCL0_Touch)
- net T0: now also U4.13 (13_LED_SCK0); no longer U4.14 (14_A0_SCK)
- net T1: now also U4.14 (14_A0_SCK); no longer U4.15 (15_A1_CS_Touch)
- net T2: now also U4.15 (15_A1_CS_Touch); no longer U4.16 (16_A2_SCL0_Touch)
- net XCTRL: now also RV2.2, U4.17 (17_A3_SDA0_Touch); no longer RV4.2, U4.23 (23_A9_Touch_PWM)
Changed lines of the file:
@@
 Wire Wire Line
 	13900 4100 13950 4100
+Text GLabel 13750 4300 3    50   Input ~ 0
+MIN_DENS
+Text GLabel 14600 4300 3    50   Input ~ 0
+MAX_DENS
+Wire Wire Line
+	11900 4250 11900 4300
+Wire Wire Line
+	12850 4250 12850 4300
 Text GLabel 11900 4300 3    50   Input ~ 0
-MIN_DENS
-Text GLabel 12850 4300 3    50   Input ~ 0
-MAX_DENS
-Wire Wire Line
-	11900 4250 11900 4300
-Wire Wire Line
-	12850 4250 12850 4300
-Text GLabel 13750 4300 3    50   Input ~ 0
 ROC
 Wire Wire Line
@@
 P 13750 4100
 F 0 "RV3" V 13543 4100 50  0000 C CNN
-F 1 "CHANGE_RATE" V 13634 4100 50  0000 C CNN
+F 1 "MIN_DENS" V 13634 4100 50  0000 C CNN
 F 2 "Crossley_Footprints:SMD_TRIM_JLC" H 13750 4100 50  0001 C CNN
 F 3 "~" H 13750 4100 50  0001 C CNN
@@
 P 12850 4100
 F 0 "RV2" V 12643 4100 50  0000 C CNN
-F 1 "MAX_DENS" V 12734 4100 50  0000 C CNN
+F 1 "XCTRL" V 12734 4100 50  0000 C CNN
 F 2 "Crossley_Footprints:SMD_TRIM_JLC" H 12850 4100 50  0001 C CNN
 F 3 "~" H 12850 4100 50  0001 C CNN
@@
 P 11900 4100
 F 0 "RV1" V 11693 4100 50  0000 C CNN
-F 1 "MIN_DENS" V 11784 4100 50  0000 C CNN
+F 1 "ROC" V 11784 4100 50  0000 C CNN
 F 2 "Crossley_Footprints:SMD_TRIM_JLC" H 11900 4100 50  0001 C CNN
 F 3 "~" H 11900 4100 50  0001 C CNN
@@
 Text GLabel 8850 2500 0    50   UnSpc ~ 0
 T3
-Text GLabel 11100 2900 2    50   UnSpc ~ 0
+Text GLabel 11100 3000 2    50   UnSpc ~ 0
 T2
-Text GLabel 11100 3000 2    50   UnSpc ~ 0
+Text GLabel 11100 3100 2    50   UnSpc ~ 0
 T1
-Text GLabel 11100 3100 2    50   UnSpc ~ 0
+Text GLabel 8850 3100 0    50   UnSpc ~ 0
 T0
 Text GLabel 8850 2000 0    50   UnSpc ~ 0
@@
 Wire Wire Line
 	8700 1200 8900 1200
-Text GLabel 8850 3100 0    50   Input ~ 0
+Text GLabel 11100 2500 2    50   Input ~ 0
 DROP
 Wire Wire Line
 	8850 3100 8900 3100
-Text GLabel 11100 2800 2    50   Input ~ 0
+Text GLabel 11100 2700 2    50   Input ~ 0
 MIN_DENS
 Wire Wire Line
 	11050 2800 11100 2800
-Text GLabel 11100 2700 2    50   Input ~ 0
+Text GLabel 11100 2600 2    50   Input ~ 0
 MAX_DENS
 Wire Wire Line
 	11050 2700 11100 2700
-Text GLabel 11100 2600 2    50   Input ~ 0
+Text GLabel 11100 2900 2    50   Input ~ 0
 ROC
 Wire Wire Line
@@
 Wire Wire Line
 	13900 9050 13900 9100
-Text GLabel 11100 2500 2    50   Input ~ 0
+Text GLabel 11100 2400 2    50   Input ~ 0
 DENS_CV
 Wire Wire Line
 	11050 2500 11100 2500
-Text GLabel 11100 2400 2    50   Input ~ 0
+Text GLabel 11100 2300 2    50   Input ~ 0
 PANIC
 Wire Wire Line
 	11050 2400 11100 2400
-Text GLabel 11100 2300 2    50   Input ~ 0
+Text GLabel 11100 2200 2    50   Input ~ 0
 DENS_IND
 Wire Wire Line
@@
 Wire Wire Line
 	14750 4100 14800 4100
-Text GLabel 14600 4300 3    50   Input ~ 0
+Text GLabel 12850 4300 3    50   Input ~ 0
 XCTRL
 Wire Wire Line
@@
 P 14600 4100
 F 0 "RV4" V 14393 4100 50  0000 C CNN
-F 1 "XCTRL" V 14484 4100 50  0000 C CNN
+F 1 "MAX_DENS" V 14484 4100 50  0000 C CNN
 F 2 "Crossley_Footprints:SMD_TRIM_JLC" H 14600 4100 50  0001 C CNN
 F 3 "~" H 14600 4100 50  0001 C CNN
@@
 	0    -1   1    0
 $EndComp
-Text GLabel 11100 2200 2    50   Input ~ 0
+Text GLabel 11100 2800 2    50   Input ~ 0
 XCTRL
 Wire Wire Line
