File: Wasp_Hive.sch (KiCad schematic (older format))
At the start: 157 parts, among them J0 WASP_OUT, J1 WASP_OUT, J10 WASP_OUT, J11 WASP_OUT, J12 WASP_OUT, J13 WASP_OUT, J14 WASP_OUT, J15 WASP_OUT, J16 DENS_OUT, J17 DENS_IN, J18 DROP_OUT, J19 PANIC_IN, J2 WASP_OUT, J20 GND, J21 GND, J22 GND, J23 GND, J24 GND, J25 PWR, J26 GND, J27 GND, J3 WASP_OUT, J4 WASP_OUT, J5 WASP_OUT, J6 WASP_OUT, J7 WASP_OUT, J8 WASP_OUT, J9 WASP_OUT, Q1 MMBT3904, Q2 MMBT3904, SW1 SW_SPDT, U0 74HC245, U1 74HC245, U2 MCP6002-xP, U3 MCP6002-xP, U4 TEENSY_3.2_MINIMAL, U5 L78M05ABDT-TR

Commit message: autorouter method
Parts:
- J0, J1, J10, J11, J12, J13, J14, J15, J2, J3, J4, J5, J6, J7, J8, J9: footprint HammerheadAudio:EuroJack_Hex_SmallHoles_NoSilk -> HammerheadAudio:EuroJack_Hex_SmallHoles_NoSilk_Clearance
Changed lines of the file:
@@
 F 0 "J15" H 5628 8825 50  0000 C CNN
 F 1 "WASP_OUT" H 5628 8734 50  0000 C CNN
-F 2 "HammerheadAudio:EuroJack_Hex_SmallHoles_NoSilk" H 5600 8600 50  0001 C CNN
+F 2 "HammerheadAudio:EuroJack_Hex_SmallHoles_NoSilk_Clearance" H 5600 8600 50  0001 C CNN
 F 3 "~" H 5600 8600 50  0001 C CNN
 	1    5600 8600
@@
 F 0 "J14" H 5628 7325 50  0000 C CNN
 F 1 "WASP_OUT" H 5628 7234 50  0000 C CNN
-F 2 "HammerheadAudio:EuroJack_Hex_SmallHoles_NoSilk" H 5600 7100 50  0001 C CNN
+F 2 "HammerheadAudio:EuroJack_Hex_SmallHoles_NoSilk_Clearance" H 5600 7100 50  0001 C CNN
 F 3 "~" H 5600 7100 50  0001 C CNN
 	1    5600 7100
@@
 F 0 "J13" H 5628 5825 50  0000 C CNN
 F 1 "WASP_OUT" H 5628 5734 50  0000 C CNN
-F 2 "HammerheadAudio:EuroJack_Hex_SmallHoles_NoSilk" H 5600 5600 50  0001 C CNN
+F 2 "HammerheadAudio:EuroJack_Hex_SmallHoles_NoSilk_Clearance" H 5600 5600 50  0001 C CNN
 F 3 "~" H 5600 5600 50  0001 C CNN
 	1    5600 5600
@@
 F 0 "J12" H 5628 4325 50  0000 C CNN
 F 1 "WASP_OUT" H 5628 4234 50  0000 C CNN
-F 2 "HammerheadAudio:EuroJack_Hex_SmallHoles_NoSilk" H 5600 4100 50  0001 C CNN
+F 2 "HammerheadAudio:EuroJack_Hex_SmallHoles_NoSilk_Clearance" H 5600 4100 50  0001 C CNN
 F 3 "~" H 5600 4100 50  0001 C CNN
 	1    5600 4100
@@
 F 0 "J11" H 4328 8775 50  0000 C CNN
 F 1 "WASP_OUT" H 4328 8684 50  0000 C CNN
-F 2 "HammerheadAudio:EuroJack_Hex_SmallHoles_NoSilk" H 4300 8550 50  0001 C CNN
+F 2 "HammerheadAudio:EuroJack_Hex_SmallHoles_NoSilk_Clearance" H 4300 8550 50  0001 C CNN
 F 3 "~" H 4300 8550 50  0001 C CNN
 	1    4300 8550
@@
 F 0 "J10" H 4328 7275 50  0000 C CNN
 F 1 "WASP_OUT" H 4328 7184 50  0000 C CNN
-F 2 "HammerheadAudio:EuroJack_Hex_SmallHoles_NoSilk" H 4300 7050 50  0001 C CNN
+F 2 "HammerheadAudio:EuroJack_Hex_SmallHoles_NoSilk_Clearance" H 4300 7050 50  0001 C CNN
 F 3 "~" H 4300 7050 50  0001 C CNN
 	1    4300 7050
@@
 F 0 "J9" H 4328 5775 50  0000 C CNN
 F 1 "WASP_OUT" H 4328 5684 50  0000 C CNN
-F 2 "HammerheadAudio:EuroJack_Hex_SmallHoles_NoSilk" H 4300 5550 50  0001 C CNN
+F 2 "HammerheadAudio:EuroJack_Hex_SmallHoles_NoSilk_Clearance" H 4300 5550 50  0001 C CNN
 F 3 "~" H 4300 5550 50  0001 C CNN
 	1    4300 5550
@@
 F 0 "J8" H 4328 4275 50  0000 C CNN
 F 1 "WASP_OUT" H 4328 4184 50  0000 C CNN
-F 2 "HammerheadAudio:EuroJack_Hex_SmallHoles_NoSilk" H 4300 4050 50  0001 C CNN
+F 2 "HammerheadAudio:EuroJack_Hex_SmallHoles_NoSilk_Clearance" H 4300 4050 50  0001 C CNN
 F 3 "~" H 4300 4050 50  0001 C CNN
 	1    4300 4050
@@
 F 0 "J7" H 2778 8775 50  0000 C CNN
 F 1 "WASP_OUT" H 2778 8684 50  0000 C CNN
-F 2 "HammerheadAudio:EuroJack_Hex_SmallHoles_NoSilk" H 2750 8550 50  0001 C CNN
+F 2 "HammerheadAudio:EuroJack_Hex_SmallHoles_NoSilk_Clearance" H 2750 8550 50  0001 C CNN
 F 3 "~" H 2750 8550 50  0001 C CNN
 	1    2750 8550
@@
 F 0 "J6" H 2778 7275 50  0000 C CNN
 F 1 "WASP_OUT" H 2778 7184 50  0000 C CNN
-F 2 "HammerheadAudio:EuroJack_Hex_SmallHoles_NoSilk" H 2750 7050 50  0001 C CNN
+F 2 "HammerheadAudio:EuroJack_Hex_SmallHoles_NoSilk_Clearance" H 2750 7050 50  0001 C CNN
 F 3 "~" H 2750 7050 50  0001 C CNN
 	1    2750 7050
@@
 F 0 "J5" H 2778 5775 50  0000 C CNN
 F 1 "WASP_OUT" H 2778 5684 50  0000 C CNN
-F 2 "HammerheadAudio:EuroJack_Hex_SmallHoles_NoSilk" H 2750 5550 50  0001 C CNN
+F 2 "HammerheadAudio:EuroJack_Hex_SmallHoles_NoSilk_Clearance" H 2750 5550 50  0001 C CNN
 F 3 "~" H 2750 5550 50  0001 C CNN
 	1    2750 5550
@@
 F 0 "J4" H 2778 4275 50  0000 C CNN
 F 1 "WASP_OUT" H 2778 4184 50  0000 C CNN
-F 2 "HammerheadAudio:EuroJack_Hex_SmallHoles_NoSilk" H 2750 4050 50  0001 C CNN
+F 2 "HammerheadAudio:EuroJack_Hex_SmallHoles_NoSilk_Clearance" H 2750 4050 50  0001 C CNN
 F 3 "~" H 2750 4050 50  0001 C CNN
 	1    2750 4050
@@
 F 0 "J3" H 1478 8725 50  0000 C CNN
 F 1 "WASP_OUT" H 1478 8634 50  0000 C CNN
-F 2 "HammerheadAudio:EuroJack_Hex_SmallHoles_NoSilk" H 1450 8500 50  0001 C CNN
+F 2 "HammerheadAudio:EuroJack_Hex_SmallHoles_NoSilk_Clearance" H 1450 8500 50  0001 C CNN
 F 3 "~" H 1450 8500 50  0001 C CNN
 	1    1450 8500
@@
 F 0 "J2" H 1478 7225 50  0000 C CNN
 F 1 "WASP_OUT" H 1478 7134 50  0000 C CNN
-F 2 "HammerheadAudio:EuroJack_Hex_SmallHoles_NoSilk" H 1450 7000 50  0001 C CNN
+F 2 "HammerheadAudio:EuroJack_Hex_SmallHoles_NoSilk_Clearance" H 1450 7000 50  0001 C CNN
 F 3 "~" H 1450 7000 50  0001 C CNN
 	1    1450 7000
@@
 F 0 "J1" H 1478 5725 50  0000 C CNN
 F 1 "WASP_OUT" H 1478 5634 50  0000 C CNN
-F 2 "HammerheadAudio:EuroJack_Hex_SmallHoles_NoSilk" H 1450 5500 50  0001 C CNN
+F 2 "HammerheadAudio:EuroJack_Hex_SmallHoles_NoSilk_Clearance" H 1450 5500 50  0001 C CNN
 F 3 "~" H 1450 5500 50  0001 C CNN
 	1    1450 5500
@@
 F 0 "J0" H 1478 4225 50  0000 C CNN
 F 1 "WASP_OUT" H 1478 4134 50  0000 C CNN
-F 2 "HammerheadAudio:EuroJack_Hex_SmallHoles_NoSilk" H 1450 4000 50  0001 C CNN
+F 2 "HammerheadAudio:EuroJack_Hex_SmallHoles_NoSilk_Clearance" H 1450 4000 50  0001 C CNN
 F 3 "~" H 1450 4000 50  0001 C CNN
 	1    1450 4000

Commit message: not working
Parts:
- J0, J1, J10, J11, J12, J13, J14, J15, J2, J3, J4, J5, J6, J7, J8, J9: footprint HammerheadAudio:EuroJack_Hex_SmallHoles_NoSilk_Clearance -> HammerheadAudio:EuroJack_Hex_SmallHoles_NoSilk_Clearance2
Changed lines of the file:
@@
 F 0 "J15" H 5628 8825 50  0000 C CNN
 F 1 "WASP_OUT" H 5628 8734 50  0000 C CNN
-F 2 "HammerheadAudio:EuroJack_Hex_SmallHoles_NoSilk_Clearance" H 5600 8600 50  0001 C CNN
+F 2 "HammerheadAudio:EuroJack_Hex_SmallHoles_NoSilk_Clearance2" H 5600 8600 50  0001 C CNN
 F 3 "~" H 5600 8600 50  0001 C CNN
 	1    5600 8600
@@
 F 0 "J14" H 5628 7325 50  0000 C CNN
 F 1 "WASP_OUT" H 5628 7234 50  0000 C CNN
-F 2 "HammerheadAudio:EuroJack_Hex_SmallHoles_NoSilk_Clearance" H 5600 7100 50  0001 C CNN
+F 2 "HammerheadAudio:EuroJack_Hex_SmallHoles_NoSilk_Clearance2" H 5600 7100 50  0001 C CNN
 F 3 "~" H 5600 7100 50  0001 C CNN
 	1    5600 7100
@@
 F 0 "J13" H 5628 5825 50  0000 C CNN
 F 1 "WASP_OUT" H 5628 5734 50  0000 C CNN
-F 2 "HammerheadAudio:EuroJack_Hex_SmallHoles_NoSilk_Clearance" H 5600 5600 50  0001 C CNN
+F 2 "HammerheadAudio:EuroJack_Hex_SmallHoles_NoSilk_Clearance2" H 5600 5600 50  0001 C CNN
 F 3 "~" H 5600 5600 50  0001 C CNN
 	1    5600 5600
@@
 F 0 "J12" H 5628 4325 50  0000 C CNN
 F 1 "WASP_OUT" H 5628 4234 50  0000 C CNN
-F 2 "HammerheadAudio:EuroJack_Hex_SmallHoles_NoSilk_Clearance" H 5600 4100 50  0001 C CNN
+F 2 "HammerheadAudio:EuroJack_Hex_SmallHoles_NoSilk_Clearance2" H 5600 4100 50  0001 C CNN
 F 3 "~" H 5600 4100 50  0001 C CNN
 	1    5600 4100
@@
 F 0 "J11" H 4328 8775 50  0000 C CNN
 F 1 "WASP_OUT" H 4328 8684 50  0000 C CNN
-F 2 "HammerheadAudio:EuroJack_Hex_SmallHoles_NoSilk_Clearance" H 4300 8550 50  0001 C CNN
+F 2 "HammerheadAudio:EuroJack_Hex_SmallHoles_NoSilk_Clearance2" H 4300 8550 50  0001 C CNN
 F 3 "~" H 4300 8550 50  0001 C CNN
 	1    4300 8550
@@
 F 0 "J10" H 4328 7275 50  0000 C CNN
 F 1 "WASP_OUT" H 4328 7184 50  0000 C CNN
-F 2 "HammerheadAudio:EuroJack_Hex_SmallHoles_NoSilk_Clearance" H 4300 7050 50  0001 C CNN
+F 2 "HammerheadAudio:EuroJack_Hex_SmallHoles_NoSilk_Clearance2" H 4300 7050 50  0001 C CNN
 F 3 "~" H 4300 7050 50  0001 C CNN
 	1    4300 7050
@@
 F 0 "J9" H 4328 5775 50  0000 C CNN
 F 1 "WASP_OUT" H 4328 5684 50  0000 C CNN
-F 2 "HammerheadAudio:EuroJack_Hex_SmallHoles_NoSilk_Clearance" H 4300 5550 50  0001 C CNN
+F 2 "HammerheadAudio:EuroJack_Hex_SmallHoles_NoSilk_Clearance2" H 4300 5550 50  0001 C CNN
 F 3 "~" H 4300 5550 50  0001 C CNN
 	1    4300 5550
@@
 F 0 "J8" H 4328 4275 50  0000 C CNN
 F 1 "WASP_OUT" H 4328 4184 50  0000 C CNN
-F 2 "HammerheadAudio:EuroJack_Hex_SmallHoles_NoSilk_Clearance" H 4300 4050 50  0001 C CNN
+F 2 "HammerheadAudio:EuroJack_Hex_SmallHoles_NoSilk_Clearance2" H 4300 4050 50  0001 C CNN
 F 3 "~" H 4300 4050 50  0001 C CNN
 	1    4300 4050
@@
 F 0 "J7" H 2778 8775 50  0000 C CNN
 F 1 "WASP_OUT" H 2778 8684 50  0000 C CNN
-F 2 "HammerheadAudio:EuroJack_Hex_SmallHoles_NoSilk_Clearance" H 2750 8550 50  0001 C CNN
+F 2 "HammerheadAudio:EuroJack_Hex_SmallHoles_NoSilk_Clearance2" H 2750 8550 50  0001 C CNN
 F 3 "~" H 2750 8550 50  0001 C CNN
 	1    2750 8550
@@
 F 0 "J6" H 2778 7275 50  0000 C CNN
 F 1 "WASP_OUT" H 2778 7184 50  0000 C CNN
-F 2 "HammerheadAudio:EuroJack_Hex_SmallHoles_NoSilk_Clearance" H 2750 7050 50  0001 C CNN
+F 2 "HammerheadAudio:EuroJack_Hex_SmallHoles_NoSilk_Clearance2" H 2750 7050 50  0001 C CNN
 F 3 "~" H 2750 7050 50  0001 C CNN
 	1    2750 7050
@@
 F 0 "J5" H 2778 5775 50  0000 C CNN
 F 1 "WASP_OUT" H 2778 5684 50  0000 C CNN
-F 2 "HammerheadAudio:EuroJack_Hex_SmallHoles_NoSilk_Clearance" H 2750 5550 50  0001 C CNN
+F 2 "HammerheadAudio:EuroJack_Hex_SmallHoles_NoSilk_Clearance2" H 2750 5550 50  0001 C CNN
 F 3 "~" H 2750 5550 50  0001 C CNN
 	1    2750 5550
@@
 F 0 "J4" H 2778 4275 50  0000 C CNN
 F 1 "WASP_OUT" H 2778 4184 50  0000 C CNN
-F 2 "HammerheadAudio:EuroJack_Hex_SmallHoles_NoSilk_Clearance" H 2750 4050 50  0001 C CNN
+F 2 "HammerheadAudio:EuroJack_Hex_SmallHoles_NoSilk_Clearance2" H 2750 4050 50  0001 C CNN
 F 3 "~" H 2750 4050 50  0001 C CNN
 	1    2750 4050
@@
 F 0 "J3" H 1478 8725 50  0000 C CNN
 F 1 "WASP_OUT" H 1478 8634 50  0000 C CNN
-F 2 "HammerheadAudio:EuroJack_Hex_SmallHoles_NoSilk_Clearance" H 1450 8500 50  0001 C CNN
+F 2 "HammerheadAudio:EuroJack_Hex_SmallHoles_NoSilk_Clearance2" H 1450 8500 50  0001 C CNN
 F 3 "~" H 1450 8500 50  0001 C CNN
 	1    1450 8500
@@
 F 0 "J2" H 1478 7225 50  0000 C CNN
 F 1 "WASP_OUT" H 1478 7134 50  0000 C CNN
-F 2 "HammerheadAudio:EuroJack_Hex_SmallHoles_NoSilk_Clearance" H 1450 7000 50  0001 C CNN
+F 2 "HammerheadAudio:EuroJack_Hex_SmallHoles_NoSilk_Clearance2" H 1450 7000 50  0001 C CNN
 F 3 "~" H 1450 7000 50  0001 C CNN
 	1    1450 7000
@@
 F 0 "J1" H 1478 5725 50  0000 C CNN
 F 1 "WASP_OUT" H 1478 5634 50  0000 C CNN
-F 2 "HammerheadAudio:EuroJack_Hex_SmallHoles_NoSilk_Clearance" H 1450 5500 50  0001 C CNN
+F 2 "HammerheadAudio:EuroJack_Hex_SmallHoles_NoSilk_Clearance2" H 1450 5500 50  0001 C CNN
 F 3 "~" H 1450 5500 50  0001 C CNN
 	1    1450 5500
@@
 F 0 "J0" H 1478 4225 50  0000 C CNN
 F 1 "WASP_OUT" H 1478 4134 50  0000 C CNN
-F 2 "HammerheadAudio:EuroJack_Hex_SmallHoles_NoSilk_Clearance" H 1450 4000 50  0001 C CNN
+F 2 "HammerheadAudio:EuroJack_Hex_SmallHoles_NoSilk_Clearance2" H 1450 4000 50  0001 C CNN
 F 3 "~" H 1450 4000 50  0001 C CNN
 	1    1450 4000
