File: Wasp_Hive.sch (KiCad schematic (older format))
At the start: 157 parts, among them J0 WASP_OUT, J1 WASP_OUT, J10 WASP_OUT, J11 WASP_OUT, J12 WASP_OUT, J13 WASP_OUT, J14 WASP_OUT, J15 WASP_OUT, J16 DENS_OUT, J17 DENS_IN, J18 DROP_OUT, J19 PANIC_IN, J2 WASP_OUT, J20 GND, J21 GND, J22 GND, J23 GND, J24 GND, J25 PWR, J26 GND, J27 GND, J3 WASP_OUT, J4 WASP_OUT, J5 WASP_OUT, J6 WASP_OUT, J7 WASP_OUT, J8 WASP_OUT, J9 WASP_OUT, Q1 MMBT3904, Q2 MMBT3904, SW1 SW_SPDT, U0 74HC245, U1 74HC245, U2 MCP6002-xP, U3 MCP6002-xP, U4 TEENSY_3.2_MINIMAL, U5 L78M05ABDT-TR

Commit message: schematic
Parts:
- R0, R12, R15, R18, R21, R24, R27, R3, R30, R33, R36, R39, R42, R45, R6, R9: value LRV_R -> LRV_R_470
- R1, R10, R13, R16, R19, R22, R25, R28, R31, R34, R37, R4, R40, R43, R46, R59, R66, R7: value WSP_R -> WSP_R_470
- R11, R14, R17, R2, R20, R23, R26, R29, R32, R35, R38, R41, R44, R47, R5, R8: value O_R -> O_R_1k
- R58, R64, R65: value DENS_R -> DENS_R_2k
- R62: value GP_R -> GP_R_100R
